File: V1/ESP-relay-8ch-V1.kicad_pcb (KiCad board)
At the start: 2 copper layers, 173 x 67.8 mm, 110 parts, among them J1 POWER & INPUTS, J2 OUT1, J3 OUT1, J4 OUT1, J5 OUT1, J6 OUT1, J7 OUT1, K1 G5PZ-1A, K2 G5PZ-1A, K3 G5PZ-1A, K4 G5PZ-1A, K5 G5PZ-1A, K6 G5PZ-1A, Q1 MMBT2222A/SOT-23-3, Q2 MMBT2222A/SOT-23-3, Q3 MMBT2222A/SOT-23-3, Q4 MMBT2222A/SOT-23-3, Q5 MMBT2222A/SOT-23-3, Q6 MMBT2222A/SOT-23-3, U1 L78M05/TO-252-2, U2 Olimex_ESP32-POE, U3 WeMos_D1_mini, U4 LTV-817S, U5 LTV-817S, U6 LTV-817S, U7 LTV-817S, U8 LTV-817S, U9 LTV-817S

Commit message: SCH and PCB updates
Parts:
- removed the D24 at (79.6, 101.6)
- removed the R31 at (76.6, 106.7)
- removed the R32 at (72.7, 109.2)
- removed the R33 at (72.7, 106.7)
- added C10: 33nF/50V/0805, Tales:C_0805_2012Metric, F.Cu at (112.1, 106.7)
- added C11: 0,1uF/50V/0805, Tales:C_0805_2012Metric, F.Cu at (113.4, 39.9)
- added C12: 12pF/50V/0603, Tales:C_0603_1608Metric, F.Cu at (129.8, 32.7)
- added C13: 10uF/16V/4x5,7, Tales:CP_Elec_4x5.7, F.Cu at (151.2, -4.27)
- added C14: 0,1uF/50V/0805, Tales:C_0805_2012Metric, F.Cu at (39.4, 85.4)
- added C15: 12pF/50V/0603, Tales:C_0603_1608Metric, F.Cu at (113.9, 48.5)
- added C16: 470uF/16V/10x10, Tales:CP_Elec_10x10, F.Cu at (74.2, 24.5)
- added D14: BLUE/0603, Tales:LED_0603_1608Metric, F.Cu at (201.4, 76.2)
- added D18: 1N4148/SOD-123, Tales:D_SOD-123, F.Cu at (202.3, 80.6)
- added D22: BLUE/0603, Tales:LED_0603_1608Metric, F.Cu at (252.2, 76.2)
- added D27: 1N4148/SOD-123, Tales:D_SOD-123, F.Cu at (253.1, 80.6)
- added D28: GREEN/0603, Tales:LED_0603_1608Metric, F.Cu at (151.6, 9.20)
- added D29: GREEN/0603, Tales:LED_0603_1608Metric, F.Cu at (159.6, 1.90)
- added J10: OUT1, Tales:TerminalBlock_Phoenix_MKDS-3-2-5.08_1x02_P5.08mm_Horizontal, F.Cu at (252.7, 118.1)
- added J2: INPUTS, Tales:TerminalBlock_Phoenix_MKDS-3-8-5.08_1x08_P5.08mm_Horizontal, F.Cu at (90.2, 118.1)
- added J6: OUT1, Tales:TerminalBlock_Phoenix_MKDS-3-2-5.08_1x02_P5.08mm_Horizontal, F.Cu at (201.9, 118.1)
- added K4: G5PZ-1A, Tales:Relay_SPST_Omron-G5PZ-1A, F.Cu at (200.7, 85.1)
- added K8: G5PZ-1A, Tales:Relay_SPST_Omron-G5PZ-1A, F.Cu at (251.5, 85.1)
- added L1: 2,2uH, Tales:L_3x3_H1.5, F.Cu at (100.3, -5.08)
- added L2: 33uH, Tales:L_12x12mm_H6mm, F.Cu at (52.1, 80.1)
- added Q4: MMBT2222A/SOT-23-3, Tales:SOT-23, F.Cu at (208.5, 80.3)
- added Q8: MMBT2222A/SOT-23-3, Tales:SOT-23, F.Cu at (258.7, 80.3)
- added R16: 3k3/0,125W/0805, Tales:R_0805_2012Metric, F.Cu at (135.5, 102.9)
- added R17: 3k3/0,125W/0805, Tales:R_0805_2012Metric, F.Cu at (135.5, 105.4)
- added R18: 3k3/0,125W/0805, Tales:R_0805_2012Metric, F.Cu at (154.0, 110.5)
- added R19: 3k3/0,125W/0805, Tales:R_0805_2012Metric, F.Cu at (154.0, 113.0)
- added R20: 5R1/0,125W/0805, Tales:R_0805_2012Metric, F.Cu at (39.4, 89.3)
- added R27: 4k7/0,125W/0805, Tales:R_0805_2012Metric, F.Cu at (201.6, 78.1)
- added R43: 10k/0,125W/0805, Tales:R_0805_2012Metric, F.Cu at (258.7, 77.5)
- added R44: 5k6/0,125W/0805, Tales:R_0805_2012Metric, F.Cu at (142.9, 10.8)
- added R48: 1k/0,125W/0805, Tales:R_0805_2012Metric, F.Cu at (258.7, 74.9)
- added R49: 820R/0,125W/0805, Tales:R_0805_2012Metric, F.Cu at (159.7, -0.87)
- added R50: 330R/0,125W/0805, Tales:R_0805_2012Metric, F.Cu at (109.7, 48.8)
- added RV4: 250VAC, Tales:RV_Disc_D12mm_W3.9mm_P7.5mm, F.Cu at (200.7, 109.2)
- added RV8: 250VAC, Tales:RV_Disc_D12mm_W3.9mm_P7.5mm, F.Cu at (251.5, 109.2)
- added U10: TX4138, Package_SO:SOIC-8-1EP_3.9x4.9mm_P1.27mm_EP2.41x3.81mm_ThermalVias, F.Cu at (34.9, 87.6)
- added U2: LTV-817S, Package_DIP:SMDIP-4_W9.53mm, F.Cu at (100.0, 86.4)
- C1: value 47uF/35V/6,3x5,4 -> 10uF/16V/4x5,7; footprint Tales:CP_Elec_6.3x5.4 -> Tales:CP_Elec_4x5.7
- C2: value 0,33uF/35V -> 47uF/35V/6,3x5,4; footprint Tales:CP_EIA-3216-18_Kemet-A_Pad1.58x1.35mm_HandSolder -> Tales:CP_Elec_6.3x5.4
- C3: value 0,1uF/50V/0805 -> 33nF/50V/0805
- D10: value 9V1/500mW -> SS510; footprint Tales:D_MiniMELF -> Tales:D_SMA
- D2, D3, D4: value GREEN/0603 -> 9V1/500mW; footprint Tales:LED_0603_1608Metric -> Tales:D_MiniMELF
- D23: value 7V5/5W/SMB -> GREEN/0603; footprint Tales:D_SMB -> Tales:LED_0603_1608Metric
- J1: value POWER & INPUTS -> +24VDC; footprint Tales:TerminalBlock_Phoenix_MKDS-3-8-5.08_1x08_P5.08mm_Horizontal -> Tales:TerminalBlock_Phoenix_MKDS-3-2-5.08_1x02_P5.08mm_Horizontal
- R1: value 270R/0,125W/0805 -> 1k2/0,125W/0805
- R10: value 1k2/0,125W/0805 -> 300k/0,125W/0805
- R11: value 3k3/0,125W/0805 -> 57,6k/0,125W/0805
- R12, R14: value 1k2/0,125W/0805 -> 3k3/0,125W/0805
- R2: value 3k9/0,125W/0805 -> 1k2/0,125W/0805
- R28: value 56R/0,125W/0805 -> 10k/0,125W/0805
- R29: value 56R/0,125W/0805 -> 300k/0,125W/0805
- R3: value 680R/0,125W/0805 -> 1k2/0,125W/0805
- R30: value 56R/0,125W/0805 -> 57,6k/0,125W/0805
- R34: value 56R/0,125W/0805 -> 1k/0,125W/0805
- R35: value 56R/0,125W/0805 -> 4k7/0,125W/0805
- R5, R7: value 3k3/0,125W/0805 -> 1k2/0,125W/0805
- R9: value 3k3/0,125W/0805 -> 30mR/0,250W/0805
- U1: value L78M05/TO-252-2 -> SY8089A1AAC; footprint Tales:TO-252-2 -> Package_TO_SOT_SMD:TSOT-23-5
- U11: renamed from U2; footprint Tales:Olimex_ESP32-POE_Pads -> Tales:Olimex_ESP32-POE
- U3: value WeMos_D1_mini -> LTV-817S; footprint Tales:WEMOS_D1_mini_light_pads -> Package_DIP:SMDIP-4_W9.53mm
- U4, U5, U6, U7, U8, U9: footprint Tales:SMDIP-4_W9.53mm -> Package_DIP:SMDIP-4_W9.53mm
- moved R34 143.8 mm to (208.6, 74.9)
- moved D23 139.3 mm to (164.0, -2.95)
- moved R42 135.0 mm to (252.4, 78.1)
- moved R28 132.1 mm to (208.6, 77.5), turned to 0 degrees
- moved R29 126.8 mm to (154.0, 3.48), turned to 0 degrees
- moved R35 106.8 mm to (133.8, 21.9), turned to 0 degrees
- moved REF** 92.0 mm to (48.3, 168.9)
- moved C2 83.4 mm to (125.7, 16.8)
- moved R11 81.5 mm to (144.0, 16.8), turned to 0 degrees
- moved R30 71.5 mm to (109.7, 45.9), turned to 0 degrees
- moved U1 67.3 mm to (116.4, 32.9)
- moved D10 62.5 mm to (43.2, 83.1)
- moved R14 59.2 mm to (154.0, 97.8), turned to 0 degrees
- moved R12 58.2 mm to (154.0, 92.7), turned to 0 degrees
- moved C1 57.3 mm to (96.5, 43.2)
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- renumbered D15 to D12, D19 to D13, D12 to D15, D20 to D17, D13 to D19, D17 to D20, D14 to D24, D18 to D25, D22 to D26, J2 to J3, J6 to J5, J3 to J7, J5 to J8, J7 to J9, K3 to K2, K5 to K3, K2 to K5, K4 to K6, K6 to K7, Q3 to Q2, Q5 to Q3, Q2 to Q5, Q4 to Q6, Q6 to Q7, R17 to R21, R36 to R22, R21 to R23, R38 to R24, R40 to R26, R16 to R31, R20 to R32, R24 to R33, R19 to R36, R23 to R38, R27 to R40, R18 to R45, R22 to R46, R26 to R47, RV3 to RV2, RV5 to RV3, RV2 to RV5, RV4 to RV6, RV6 to RV7
Connections:
- C1 pad 1: +VReg -> +5V
- C3 pad 1: +5V -> Net-(C3-Pad1)
- D1 pad 1: Net-(D1-Pad1) -> +VReg
- D10 pad 1: Net-(C9-Pad1) -> Net-(C14-Pad2)
- D10 pad 2: Net-(D10-Pad2) -> GNDREF
- D2 pad 1: GNDREF -> Net-(C3-Pad1)
- D23 pad 1: +VReg -> GNDREF
- D3 pad 1: GNDREF -> Net-(C4-Pad1)
- D4 pad 1: GNDREF -> Net-(C5-Pad1)
- D5 pad 1: Net-(C4-Pad1) -> Net-(C6-Pad1)
- D6 pad 1: Net-(C5-Pad1) -> Net-(C7-Pad1)
- D7 pad 1: Net-(C6-Pad1) -> Net-(C8-Pad1)
- D8 pad 1: Net-(C7-Pad1) -> Net-(C9-Pad1)
- D9 pad 1: Net-(C8-Pad1) -> Net-(C10-Pad1)
- R1 pad 1: +3V3 -> Net-(C3-Pad1)
- R1 pad 2: Net-(D2-Pad2) -> Net-(J2-Pad1)
- R10 pad 1: Net-(C7-Pad1) -> +3.3V
- R10 pad 2: Net-(J1-Pad6) -> Net-(C12-Pad2)
- R11 pad 1: +3V3 -> Net-(C12-Pad2)
- R11 pad 2: IN4 -> GNDREF
- R12 pad 1: Net-(C8-Pad1) -> +3.3V
- R12 pad 2: Net-(J1-Pad7) -> IN1
- R13 pad 1: +3V3 -> +3.3V
- R13 pad 2: IN5 -> IN2
- R14 pad 1: Net-(C9-Pad1) -> +3.3V
- R14 pad 2: Net-(J1-Pad8) -> IN3
- R15 pad 1: +3V3 -> +3.3V
- R15 pad 2: IN6 -> IN4
- R2 pad 1: +VReg -> Net-(C4-Pad1)
- R2 pad 2: Net-(D3-Pad2) -> Net-(J2-Pad2)
- R24 pad 1: OUT3 -> OUT2
- R26 pad 1: OUT5 -> OUT3
- R28 pad 1: Net-(D1-Pad1) -> OUT4
- R28 pad 2: Net-(R28-Pad2) -> GNDREF
- R29 pad 1: Net-(D1-Pad1) -> +5V
- R29 pad 2: Net-(R29-Pad2) -> Net-(C15-Pad2)
- R3 pad 1: +5V -> Net-(C5-Pad1)
- R3 pad 2: Net-(D4-Pad2) -> Net-(J2-Pad3)
- R30 pad 1: Net-(R28-Pad2) -> Net-(C15-Pad2)
- R30 pad 2: Net-(R30-Pad2) -> GNDREF
- R32 pad 2: OUT3 -> OUT2
- R33 pad 2: OUT5 -> OUT3
- R34 pad 2: +VReg -> OUT4
- R35 pad 1: Net-(R33-Pad2) -> +3.3V
- R35 pad 2: +VReg -> Net-(R35-Pad2)
- R37 pad 1: OUT2 -> OUT5
- R39 pad 1: OUT4 -> OUT6
- R4 pad 1: Net-(C4-Pad1) -> Net-(C6-Pad1)
- R4 pad 2: Net-(J1-Pad3) -> Net-(J2-Pad4)
- R41 pad 1: OUT6 -> OUT7
- R42 pad 1: +3V3 -> +24V
- R42 pad 2: Net-(R42-Pad2) -> Net-(D22-Pad2)
- R45 pad 2: OUT2 -> OUT5
- R46 pad 2: OUT4 -> OUT6
- R47 pad 2: OUT6 -> OUT7
- R5 pad 1: +3V3 -> Net-(C7-Pad1)
- R5 pad 2: IN1 -> Net-(J2-Pad5)
- R6 pad 1: Net-(C5-Pad1) -> Net-(C8-Pad1)
- R6 pad 2: Net-(J1-Pad4) -> Net-(J2-Pad6)
- R7 pad 1: +3V3 -> Net-(C9-Pad1)
- R7 pad 2: IN2 -> Net-(J2-Pad7)
- R8 pad 1: Net-(C6-Pad1) -> Net-(C10-Pad1)
- R8 pad 2: Net-(J1-Pad5) -> Net-(J2-Pad8)
- R9 pad 1: +3V3 -> +VReg
- R9 pad 2: IN3 -> Net-(R9-Pad2)
- U1 pad 1: +VReg -> +5V
- U1 pad 3: +5V -> Net-(L1-Pad1)
- U11 pad 10: unconnected-(U2-Pad10) -> OUT8
- U11 pad 12: IN6 -> IN8
- U11 pad 13: IN5 -> IN7
- U11 pad 2: +3V3 -> unconnected-(U11-Pad2)
- U11 pad 4: Net-(R42-Pad2) -> Net-(R35-Pad2)
- U11 pad 5: unconnected-(U2-Pad5) -> IN5
- U11 pad 6: unconnected-(U2-Pad6) -> IN6
- U11 pad 8: unconnected-(U2-Pad8) -> OUT7
- U3 pad 1: Net-(R42-Pad2) -> Net-(D3-Pad2)
- U3 pad 2: unconnected-(U3-Pad2) -> GNDREF
- U3 pad 3: unconnected-(U3-Pad3) -> GNDREF
- U3 pad 4: IN1 -> IN2
- U4 pad 1: Net-(D5-Pad2) -> Net-(D4-Pad2)
- U4 pad 4: IN1 -> IN3
- U5 pad 1: Net-(D6-Pad2) -> Net-(D5-Pad2)
- U5 pad 4: IN2 -> IN4
- U6 pad 1: Net-(D7-Pad2) -> Net-(D6-Pad2)
- U6 pad 4: IN3 -> IN5
- U7 pad 1: Net-(D8-Pad2) -> Net-(D7-Pad2)
- U7 pad 4: IN4 -> IN6
- U8 pad 1: Net-(D9-Pad2) -> Net-(D8-Pad2)
- U8 pad 4: IN5 -> IN7
- U9 pad 1: Net-(D10-Pad2) -> Net-(D9-Pad2)
- U9 pad 4: IN6 -> IN8
Routing:
- net GNDREF: track 437.8 -> 0.00 mm, vias 20 -> 0
- net +24V: track 282.3 -> 0.00 mm, vias 2 -> 0
- net OUT6: track 148.7 -> 0.00 mm, vias 3 -> 0
- net +3V3: track 145.0 -> 0.00 mm
- net OUT5: track 127.8 -> 0.00 mm, vias 3 -> 0
- net OUT4: track 126.0 -> 0.00 mm, vias 3 -> 0
- net +5V: track 120.8 -> 0.00 mm, vias 6 -> 0
- net OUT3: track 88.7 -> 0.00 mm, vias 3 -> 0
- net IN3: track 76.5 -> 0.00 mm, vias 3 -> 0
- net OUT2: track 75.5 -> 0.00 mm, vias 3 -> 0
- net IN4: track 63.8 -> 0.00 mm, vias 3 -> 0
- net OUT1: track 60.7 -> 0.00 mm, vias 3 -> 0
- net Net-(J1-Pad3): track 56.2 -> 0.00 mm
- net IN1: track 55.4 -> 0.00 mm, vias 2 -> 0
- net Net-(R42-Pad2): track 55.3 -> 0.00 mm, vias 2 -> 0
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Other:
- board text added: "8x IN 24VDC/8x OUT RLY"
- board text added: "ESP-RELAY-8CH-V1"
- board text removed: "6x IN 24VDC/6x OUT RLY"
- board text removed: "ESP-RELAY-6CH-V2"
- board text removed: "WEMOS D1 MINI"

Commit message: SCH and PCB updates
Parts:
- moved R29 137.6 mm to (68.2, 111.1), turned to 180 degrees
- moved C13 113.6 mm to (73.8, 78.7)
- moved R49 94.1 mm to (100.6, 72.4)
- moved D23 93.3 mm to (104.9, 69.2), turned to 180 degrees
- moved D29 91.7 mm to (104.9, 75.6), turned to 180 degrees
- moved C2 90.7 mm to (71.5, 89.5)
- moved L1 83.6 mm to (70.5, 73.0), turned to 180 degrees
- moved R11 81.2 mm to (80.9, 67.9)
- moved D28 78.5 mm to (104.9, 72.4), turned to 180 degrees
- moved R35 78.5 mm to (135.5, 100.3), turned to 180 degrees
- moved C15 76.0 mm to (68.1, 109.2), turned to 180 degrees
- moved R30 74.1 mm to (68.2, 107.3)
- moved R44 72.1 mm to (100.6, 69.2)
- moved C11 70.2 mm to (69.5, 94.6)
- moved C16 65.7 mm to (83.4, 89.5), turned to 180 degrees
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Routing:
- net GNDREF: track 0.00 -> 189.7 mm, vias 0 -> 8
- net Net-(C3-Pad1): track 0.00 -> 36.5 mm, vias 0 -> 2
- net Net-(C7-Pad1): track 0.00 -> 31.3 mm, vias 0 -> 2
- net Net-(C4-Pad1): track 0.00 -> 24.2 mm, vias 0 -> 2
- net Net-(C8-Pad1): track 0.00 -> 22.9 mm, vias 0 -> 2
- net Net-(C9-Pad1): track 0.00 -> 18.7 mm, vias 0 -> 2
- net Net-(C5-Pad1): track 0.00 -> 17.4 mm, vias 0 -> 2
- net Net-(C10-Pad1): track 0.00 -> 17.0 mm
- net Net-(C6-Pad1): track 0.00 -> 15.8 mm
- net +3.3V: track 0.00 -> 15.2 mm
- net Net-(J2-Pad8): track 0.00 -> 7.62 mm
- net Net-(J2-Pad7): track 0.00 -> 7.62 mm
- net Net-(J2-Pad6): track 0.00 -> 7.62 mm
- net Net-(J2-Pad5): track 0.00 -> 7.62 mm
- net Net-(J2-Pad4): track 0.00 -> 7.62 mm
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
Commit message: SCH and PCB development
Parts:
- C1, C13: value 10uF/16V/4x5,7 -> 10uF/16V/1206; footprint Tales:CP_Elec_4x5.7 -> Tales:C_1206_3216Metric
- C12: value 12pF/50V/0603 -> 22pF/50V/0603
- R10: value 300k/0,125W/0805 -> 100k/0,125W/0805
- R11: value 57,6k/0,125W/0805 -> 22,1k/0,125W/0805
- U1: footprint Package_TO_SOT_SMD:TSOT-23-5 -> Tales:TSOT-23-5
- U10: footprint Package_SO:SOIC-8-1EP_3.9x4.9mm_P1.27mm_EP2.41x3.81mm_ThermalVias -> Tales:SOIC-8-1EP_3.9x4.9mm_P1.27mm_EP2.29x3mm_ThermalVias
- moved REF** 134.3 mm to (144.8, 75.6)
- moved R15 57.2 mm to (106.7, 68.2), turned to -90 degrees
- moved R19 57.0 mm to (118.7, 68.2), turned to -90 degrees
- moved R14 53.7 mm to (109.2, 68.2), turned to -90 degrees
- moved R18 53.5 mm to (121.3, 68.2), turned to -90 degrees
- moved R13 50.2 mm to (111.8, 68.2), turned to -90 degrees
- moved R12 46.7 mm to (114.3, 68.2), turned to -90 degrees
- moved R17 39.0 mm to (123.8, 68.2), turned to -90 degrees
- moved R16 35.3 mm to (128.9, 68.2), turned to -90 degrees
- moved R35 33.4 mm to (126.4, 68.2), turned to -90 degrees
- moved C3 21.9 mm to (96.1, 109.5), turned to 90 degrees
- moved C7 21.9 mm to (114.4, 109.5), turned to 90 degrees
- moved C4 16.4 mm to (100.7, 109.5), turned to 90 degrees
- moved C8 16.2 mm to (119.0, 109.5), turned to 90 degrees
- moved C6 14.6 mm to (109.9, 109.5), turned to 90 degrees
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Routing:
- net GNDREF: track 189.7 -> 544.2 mm, vias 8 -> 27
- net +24V: track 5.08 -> 318.0 mm, vias 0 -> 2
- net OUT8: track 0.00 -> 181.6 mm, vias 0 -> 2
- net OUT7: track 0.00 -> 162.5 mm, vias 0 -> 2
- net OUT6: track 0.00 -> 151.1 mm, vias 0 -> 2
- net OUT5: track 0.00 -> 132.1 mm, vias 0 -> 2
- net OUT4: track 0.00 -> 127.0 mm, vias 0 -> 2
- net IN4: track 2.54 -> 110.4 mm, vias 0 -> 4
- net OUT3: track 0.00 -> 102.8 mm, vias 0 -> 2
- net IN3: track 2.54 -> 96.4 mm, vias 0 -> 5
- net +5V: track 0.00 -> 89.3 mm, vias 0 -> 2
- net IN8: track 2.54 -> 90.0 mm, vias 0 -> 5
- net OUT2: track 0.00 -> 83.8 mm, vias 0 -> 2
- net IN7: track 2.54 -> 85.1 mm, vias 0 -> 5
- net IN2: track 2.54 -> 84.9 mm, vias 0 -> 5
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- added copper zone on F.Cu, net +3.3V
- added copper zone on F.Cu, net +5V
- added copper zone on B.Cu, net GNDREF
- added copper zone on F.Cu, net GNDREF
- added copper zone on F.Cu, net Net-(C12-Pad2)
- added copper zone on F.Cu, net Net-(L1-Pad1)
Other:
- board size 173 x 67.8 mm -> 198 x 67.8 mm
- board text added: "24V"
- board text added: "3,3V"
- board text added: "5V"
- board text added: "IN7"
- board text added: "IN8"
- board text added: "OUT7"
- board text added: "OUT8"
- board text removed: "24V OK"
- board text removed: "3,3V OK"
- board text removed: "5V OK"

Commit message: SCH and PCB updates
Parts:
- moved R12 14.1 mm to (101.9, 74.9), turned to 0 degrees
- moved R18 11.2 mm to (110.1, 68.2), turned to 0 degrees
- moved R13 10.8 mm to (101.9, 72.6), turned to 0 degrees
- moved R19 8.90 mm to (110.1, 70.5), turned to 0 degrees
- moved R14 7.65 mm to (101.9, 70.4), turned to 0 degrees
- moved R35 6.71 mm to (119.7, 68.2), turned to 0 degrees
- moved D23 5.56 mm to (91.6, 74.9)
- moved D28 5.45 mm to (91.6, 71.8)
- moved D29 5.41 mm to (91.6, 68.6)
- moved R15 4.80 mm to (101.9, 68.1), turned to 0 degrees
- moved R17 4.74 mm to (119.7, 70.5), turned to 0 degrees
- moved R44 4.62 mm to (87.9, 74.9)
- moved R49 4.49 mm to (87.9, 71.8)
- moved R50 4.45 mm to (87.9, 68.6)
- moved C15 1.42 mm to (71.9, 111.8), turned to 180 degrees
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Routing:
- net GNDREF: track 544.2 -> 490.2 mm, vias 27 -> 60
- net +5V: track 89.3 -> 136.9 mm, vias 2 -> 3
- net +3.3V: track 53.6 -> 95.6 mm
- net +VReg: track 38.5 -> 58.5 mm, vias 0 -> 2
- net Net-(J9-Pad1): track 18.3 -> 36.6 mm
- net Net-(J8-Pad1): track 18.3 -> 36.6 mm
- net Net-(J6-Pad1): track 18.3 -> 36.6 mm
- net Net-(J4-Pad1): track 18.3 -> 36.6 mm
- net Net-(J3-Pad1): track 18.3 -> 36.6 mm
- net Net-(J7-Pad1): track 18.3 -> 36.6 mm
- net Net-(J5-Pad1): track 18.3 -> 36.6 mm
- net Net-(J10-Pad1): track 18.3 -> 36.6 mm
- net Net-(C14-Pad2): track 16.1 -> 0.00 mm
- net Net-(J8-Pad2): track 14.8 -> 29.5 mm
- net Net-(J7-Pad2): track 14.8 -> 29.5 mm
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- added copper zone on F.Cu, net +VReg
- added copper zone on F.Cu, net Net-(C14-Pad2)
- added copper zone on B.Cu, net Net-(R9-Pad2)
Other:
- board text added: "SUPORTES PCI METALTEX SP7 1x pé macho 9 mm 1x pé fêmea 9 mm 4x espaçadores 45 mm Comprimento total 198 mm Largura da placa 67,8 mm"
- board text removed: "SUPORTES PCI METALTEX SP7 1x pé macho 9 mm 1x pé fêmea 9 mm 1x espaçador 20 mm 3x espaçadores 45 mm Comprimento total 173 mm Largura da placa 67,8 mm"

Commit message: Update ESP-relay-8ch-V1.kicad_pcb
Parts:
- moved R12 0.63 mm to (101.2, 74.9)
- moved R13 0.63 mm to (101.2, 72.6)
- moved R14 0.63 mm to (101.2, 70.4)
- moved R15 0.63 mm to (101.2, 68.1)
- moved C9 0.06 mm to (123.6, 109.5)
Routing:
- net GNDREF: track 490.2 -> 498.0 mm, vias 60 -> 62
- net +5V: track 136.9 -> 136.0 mm
- net IN3: track 100.1 -> 100.7 mm
- net IN4: track 113.2 -> 113.8 mm
- net IN2: track 87.0 -> 87.6 mm
- net IN1: track 75.1 -> 75.7 mm

Commit message: Development
Parts:
- J10: value OUT1 -> OUT8
- J4: value OUT1 -> OUT2
- J5: value OUT1 -> OUT3
- J6: value OUT1 -> OUT4
- J7: value OUT1 -> OUT5
- J8: value OUT1 -> OUT6
- J9: value OUT1 -> OUT7
- moved DRW1 7.10 mm to (141.6, 81.9)
- moved C15 4.26 mm to (73.8, 108.0)
- moved R29 4.26 mm to (73.9, 109.9)
- moved J1 3.17 mm to (75.6, 118.1)
- moved C10 3.17 mm to (125.0, 109.5)
- moved C3 3.17 mm to (93.0, 109.5)
- moved C4 3.17 mm to (97.5, 109.5)
- moved C5 3.17 mm to (102.1, 109.5)
- moved C6 3.17 mm to (106.7, 109.5)
- moved C7 3.17 mm to (111.3, 109.5)
- moved C8 3.17 mm to (115.8, 109.5)
- moved C9 3.17 mm to (120.4, 109.5)
- moved D2 3.17 mm to (95.3, 81.8)
- moved D3 3.17 mm to (95.3, 88.1)
- moved D4 3.17 mm to (95.3, 94.5)
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- renumbered REF** to DRW1
Routing:
- net GNDREF: track 498.0 -> 518.3 mm, vias 62 -> 65
- net Net-(C14-Pad2): track 0.00 -> 13.2 mm
- net +5V: track 136.0 -> 143.8 mm
- net Net-(C12-Pad2): track 0.00 -> 7.27 mm
- net Net-(C3-Pad1): track 30.3 -> 35.2 mm
- net +3.3V: track 95.6 -> 99.0 mm
- net OUT4: track 128.1 -> 131.3 mm
- net OUT1: track 65.3 -> 68.5 mm
- net OUT8: track 178.9 -> 182.1 mm
- net OUT6: track 148.4 -> 151.6 mm
- net OUT7: track 159.8 -> 163.0 mm
- net OUT5: track 129.4 -> 132.5 mm
- net OUT3: track 104.0 -> 107.1 mm
- net OUT2: track 84.9 -> 88.1 mm
- net +VReg: track 58.5 -> 60.4 mm
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Other:
- outline, holes or cut-outs redrawn

Commit message: SCH tweaks
Routing:
- added copper zone on F.Cu, net +24V
Changed lines of the file:
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@@
   (via (at 151.135 87.63) (size 1.3) (drill 0.5) (layers "F.Cu" "B.Cu") (net 2))
   (via (at 151.135 123.19) (size 1.3) (drill 0.5) (layers "F.Cu" "B.Cu") (net 2))
-  (segment (start 151.135 123.19) (end 151.135 87.63) (width 1.016) (layer "B.Cu") (net 2))
+  (segment (start 151.135 123.19) (end 151.135 87.63) (width 1.524) (layer "B.Cu") (net 2))
   (segment (start 81.7575 76.2) (end 83.82 76.2) (width 1.016) (layer "F.Cu") (net 3))
   (segment (start 81.7575 76.2) (end 81.7575 73.025) (width 0.635) (layer "F.Cu") (net 3))
@@
         (xy 74.681 77.724)
         (xy 67.315 77.724)
-        (xy 67.315 67.31)
-        (xy 72.395 67.31)
+        (xy 67.315 69.85)
+        (xy 72.395 69.85)
       )
     )
@@
         (xy 87 82.55)
         (xy 92.08 82.55)
+      )
+    )
+  )
+  (zone (net 2) (net_name "+24V") (layer "F.Cu") (hatch edge 0.508)
+    (connect_pads yes (clearance 0.381))
+    (min_thickness 0.254) (filled_areas_thickness no)
+    (fill yes (thermal_gap 0.508) (thermal_bridge_width 0.508))
+    (polygon
+      (pts
+        (xy 77.47 120.523)
+        (xy 80.137 123.19)
+        (xy 70.993 123.19)
+        (xy 73.66 120.523)
+        (xy 73.66 116.332)
+        (xy 77.47 116.332)
       )
     )
@@
         (xy 76.586 73.914)
         (xy 72.776 73.914)
-        (xy 72.776 67.31)
-        (xy 74.681 67.31)
-      )
-    )
+        (xy 72.776 69.85)
+        (xy 74.681 69.85)
+      )
+    )
