File: V1/ESP-relay-8ch-V1.kicad_pcb (KiCad board)
At the start: 2 copper layers, 198 x 67.8 mm, 143 parts, among them J1 +24VDC, J10 OUT8, J2 INPUTS, J3 OUT1, J4 OUT2, J5 OUT3, J6 OUT4, J7 OUT5, J8 OUT6, J9 OUT7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

Commit message: Design optimization
Parts:
- removed LOGO1: Logo_Open_Hardware_Large, Symbol:OSHW-Logo2_14.6x12mm_SilkScreen
