File: V1/ESP-relay-8ch-V1.kicad_sch (KiCad schematic)
At the start: 104 parts, among them J1 POWER & INPUTS, J2 OUT1, J3 OUT1, J4 OUT1, J5 OUT1, J6 OUT1, J7 OUT1, K1 G5PZ-1A, K2 G5PZ-1A, K3 G5PZ-1A, K4 G5PZ-1A, K5 G5PZ-1A, K6 G5PZ-1A, Q1 MMBT2222A/SOT-23-3, Q2 MMBT2222A/SOT-23-3, Q3 MMBT2222A/SOT-23-3, Q4 MMBT2222A/SOT-23-3, Q5 MMBT2222A/SOT-23-3, Q6 MMBT2222A/SOT-23-3, U1 TX4138, U2 SY8089AAAC, U3 Olimex_ESP32-POE, U4 LTV-817S, U5 LTV-817S, U6 LTV-817S, U7 LTV-817S, U8 LTV-817S, U9 LTV-817S

Commit message: SCH and PCB updates
Parts:
- removed C3: 0,1uF/50V/0805, Tales:C_0805_2012Metric, symbol Device:C_Small
- added C1, C13: 10uF/16V/4x5,7, Tales:CP_Elec_4x5.7, symbol Device:C_Polarized_Small_US
- added C10, C9: 33nF/50V/0805, Tales:C_0805_2012Metric, symbol Device:C_Small
- added C12, C15: 12pF/50V/0603, Tales:C_0603_1608Metric, symbol Device:C_Small
- added C16: 470uF/16V/10x10, Tales:CP_Elec_10x10, symbol Device:C_Polarized_Small_US
- added D14, D22: BLUE/0603, Tales:LED_0603_1608Metric, symbol Device:LED
- added D18, D27: 1N4148/SOD-123, Tales:D_SOD-123, symbol Device:D
- added D8, D9: 9V1/500mW, Tales:D_MiniMELF, symbol Device:D_Zener
- added J1: +24VDC, Tales:TerminalBlock_Phoenix_MKDS-3-2-5.08_1x02_P5.08mm_Horizontal, symbol Connector_Generic:Conn_01x02
- added J10, J6: OUT1, Tales:TerminalBlock_Phoenix_MKDS-3-2-5.08_1x02_P5.08mm_Horizontal, symbol Connector_Generic:Conn_01x02
- added K4, K8: G5PZ-1A, Tales:Relay_SPST_Omron-G5PZ-1A, symbol Tales:G5PZ-1A
- added L1: 2,2uH, Tales:L_3x3_H1.5, symbol Device:L
- added Q4, Q8: MMBT2222A/SOT-23-3, Tales:SOT-23, symbol Device:Q_NPN_BEC
- added R10, R29: 300k/0,125W/0805, Tales:R_0805_2012Metric, symbol Device:R_US
- added R11, R30: 57,6k/0,125W/0805, Tales:R_0805_2012Metric, symbol Device:R_US
- added R18, R19: 3k3/0,125W/0805, Tales:R_0805_2012Metric, symbol Device:R_US
- added R27, R42: 4k7/0,125W/0805, Tales:R_0805_2012Metric, symbol Device:R_US
- added R28, R43: 10k/0,125W/0805, Tales:R_0805_2012Metric, symbol Device:R_US
- added R34, R48: 1k/0,125W/0805, Tales:R_0805_2012Metric, symbol Device:R_US
- added R7, R8: 1k2/0,125W/0805, Tales:R_0805_2012Metric, symbol Device:R_US
- added RV4, RV8: 250VAC, Tales:RV_Disc_D12mm_W3.9mm_P7.5mm, symbol Device:Varistor
- added U8, U9: LTV-817S, Package_DIP:SMDIP-4_W9.53mm, symbol Isolator:LTV-817S
- D10: renamed from D2; footprint Diode_SMD:D_SMA -> Tales:D_SMA
- J2: renamed from J1; value POWER & INPUTS -> INPUTS
- L2: renamed from L1; footprint (none) -> Tales:L_12x12mm_H6mm; Case (none) -> 12x12
- R35: renamed from R42; Mfr PN 0805W8F2700T5E -> 0805W8F4701T5E; Vendor PN C17590 -> C17673
- U1: renamed from U2; value SY8089AAAC -> SY8089A1AAC; Case (none) -> SOT-23-5; JLCPCB BOM (none) -> 1; LCSC Part (none) -> C479074; Mfr (none) -> Silergy; Mfr PN (none) -> SY8089A1AAC; Vendor (none) -> JLCPCB; Vendor PN (none) -> C479074
- U10: renamed from U1; Case (none) -> SOIC-8; JLCPCB BOM (none) -> 1; LCSC Part (none) -> C329267; Mfr (none) -> XDS; Mfr PN (none) -> TX4138; Vendor (none) -> JLCPCB; Vendor PN (none) -> C329267
- U11: renamed from U3; footprint Tales:Olimex_ESP32-POE_Pads -> Tales:Olimex_ESP32-POE
- U2: renamed from U4; footprint Tales:SMDIP-4_W9.53mm -> Package_DIP:SMDIP-4_W9.53mm
- U3: renamed from U5; footprint Tales:SMDIP-4_W9.53mm -> Package_DIP:SMDIP-4_W9.53mm
- U4: renamed from U6; footprint Tales:SMDIP-4_W9.53mm -> Package_DIP:SMDIP-4_W9.53mm
- U5: renamed from U7; footprint Tales:SMDIP-4_W9.53mm -> Package_DIP:SMDIP-4_W9.53mm
- U6: renamed from U8; footprint Tales:SMDIP-4_W9.53mm -> Package_DIP:SMDIP-4_W9.53mm
- U7: renamed from U9; footprint Tales:SMDIP-4_W9.53mm -> Package_DIP:SMDIP-4_W9.53mm
- gave numbers to parts that had none: 2
- renumbered C2 to C11, C1 to C2, C4 to C3, C5 to C4, C6 to C5, C7 to C6, C8 to C7, C9 to C8, D15 to D12, D19 to D13, D12 to D15, D20 to D17, D13 to D19, D5 to D2, D17 to D20, D3 to D23, D14 to D24, D18 to D25, D22 to D26, D4 to D28, D2 to D29, D6 to D3, D7 to D4, D8 to D5, D9 to D6, D10 to D7, J2 to J3, J6 to J5, J3 to J7, J5 to J8, J7 to J9, K3 to K2, K5 to K3, K2 to K5, K4 to K6, K6 to K7, Q3 to Q2, Q5 to Q3, Q2 to Q5, Q4 to Q6, Q6 to Q7, R4 to R1, R5 to R12, R7 to R13, R9 to R14, R11 to R15, R13 to R16, R15 to R17, R6 to R2, R17 to R21, R36 to R22, R21 to R23, R38 to R24, R40 to R26, R8 to R3, R16 to R31, R20 to R32, R24 to R33, R19 to R36, R23 to R38, R10 to R4, R27 to R40, R2 to R44, R18 to R45, R22 to R46, R26 to R47, R3 to R49, R12 to R5, R4 to R50, R14 to R6, R1 to R9, RV3 to RV2, RV5 to RV3, RV2 to RV5, RV4 to RV6, RV6 to RV7
Connections:
- net +24V: now also D18.1 (K), D27.1 (K), J1.1 (Pin_1), K4.1, K8.1, R27.1, R42.1; no longer J2.1 (Pin_1)
- net +5V: now also U1.1 (EN), U1.4 (IN), C1.1, C15.1, C16.1, R29.1
- net GNDREF: now also U1.2 (GND), C1.2, C10.2, C13.2, C16.2, C9.2, J1.2 (Pin_2), Q4.2 (E), Q8.2 (E), R11.2, R28.2, R30.2, R43.2, U8.2, U8.3, U9.2, U9.3; no longer J2.2 (Pin_2)
- net IN5: now also U11.5 (GPIO0); no longer U11.13 (GPIO15\HS2_CMD)
- net IN6: now also U11.6 (GPIO1\U0TXD); no longer U11.12 (GPIO14\HS2_CLK)
- net OUT2: now also R24.1, R32.2; no longer R37.1, R45.2
- net OUT3: now also R26.1, R33.2; no longer R24.1, R32.2
- net OUT4: now also R28.1, R34.2; no longer R39.1, R46.2
- net OUT5: now also R37.1, R45.2; no longer R26.1, R33.2
- net OUT6: now also R39.1, R46.2; no longer R41.1, R47.2
- net at R1.2: now also J2.1 (Pin_1); no longer J2.3 (Pin_3)
- net OUT8: now reaches U11.10 (GPIO5\SPI_CS)
- net OUT8: now also R43.1, R48.2
- net OUT7: now reaches U11.8 (GPIO3\U0RXD)
- net OUT7: now also R41.1, R47.2
- net at R2.2: now also J2.2 (Pin_2); no longer J2.4 (Pin_4)
- net at R3.2: now also J2.3 (Pin_3); no longer J2.5 (Pin_5)
- net at R4.2: now also J2.4 (Pin_4); no longer J2.6 (Pin_6)
- net at R5.2: now also J2.5 (Pin_5); no longer J2.7 (Pin_7)
- net at R6.2: now also J2.6 (Pin_6); no longer J2.8 (Pin_8)
- net at U10.5 (FB): now also C15.2, R29.2, R30.1
- net at U1.3 (LX): now also L1.1
- net at U1.5 (FB): now also C12.2, R10.2, R11.1
- net +3V3 renamed +3.3V
- net +3.3V: now also C12.1, C13.1, L1.2, R10.1, R18.1, R19.1; no longer U11.2 (3V3)
- new net: J2.7 (Pin_7), R7.2
- new net: J2.8 (Pin_8), R8.2
- new net: D14.2 (A), R27.2
- new net: J10.1 (Pin_1), K8.2, RV8.1
- new net: J10.2 (Pin_2), K8.3, RV8.2
- new net: Q4.1 (B), R34.1
- new net: D14.1 (K), D18.2 (A), K4.4, Q4.3 (C)
- new net: C10.1, D9.1 (K), R8.1
- new net: D9.2 (A), U9.1
- new net: J6.1 (Pin_1), K4.2, RV4.1
- new net: J6.2 (Pin_2), K4.3, RV4.2
- new net: C9.1, D8.1 (K), R7.1
- new net: D8.2 (A), U8.1
- new net: Q8.1 (B), R48.1
- new net: D22.1 (K), D27.2 (A), K8.4, Q8.3 (C)
- new net: D22.2 (A), R42.2
- new net IN7: R18.2, U11.13 (GPIO15\HS2_CMD), U8.4
- new net IN8: R19.2, U11.12 (GPIO14\HS2_CLK), U9.4
- no-connect marks 4 -> 3
Other:
- moved on the sheet: C11, C14, C2, C3, C4, C5, C6, C7, C8, D1, D10, D11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

Commit message: SCH and PCB updates
Other:
- title: ESP 6x 24VDC Input 6x Relay Output Module -> ESP 8x 24VDC Input 8x Relay Output Module
Changed lines of the file:
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@@
   (paper "A3")
   (title_block
-    (title "ESP 6x 24VDC Input 6x Relay Output Module")
-    (date "2022-10-09")
-    (rev "V3")
+    (title "ESP 8x 24VDC Input 8x Relay Output Module")
+    (date "2022-10-10")
+    (rev "V1")
   )
   (junction (at 69.85 68.58) (diameter 0) (color 0 0 0 0)

Commit message: SCH and PCB development
Parts:
- C1, C13: value 10uF/16V/4x5,7 -> 10uF/16V/1206; footprint Tales:CP_Elec_4x5.7 -> Tales:C_1206_3216Metric; Case 4x5,7 -> 1206/3216; LCSC Part C249724 -> C1849; Mfr Lelon -> Samsung; Mfr PN VEU100M1CTR-0406 -> CL31A106KOHNNNE; Technology Electrolitic -> Ceramic; Vendor PN C249724 -> C1849
- C12: value 12pF/50V/0603 -> 22pF/50V/0603; LCSC Part C38523 -> C1653; Mfr PN CL10C120JB8NNNC -> CL10C220JB8NNNC; Vendor PN C38523 -> C1653
- R10: value 300k/0,125W/0805 -> 100k/0,125W/0805; LCSC Part C17616 -> C149504; Mfr PN 0805W8F3003T5E -> 0805W8F1003T5E; Vendor PN C17616 -> C149504
- R11: value 57,6k/0,125W/0805 -> 22,1k/0,125W/0805; LCSC Part C17758 -> C17552; Mfr PN 0805W8F5762T5E -> 0805W8F2212T5E; Vendor PN C17758 -> C17552
- U1: footprint Package_TO_SOT_SMD:TSOT-23-5 -> Tales:TSOT-23-5
- U10: footprint Package_SO:SOIC-8-1EP_3.9x4.9mm_P1.27mm_EP2.41x3.81mm_ThermalVias -> Tales:SOIC-8-1EP_3.9x4.9mm_P1.27mm_EP2.29x3mm_ThermalVias
Changed lines of the file:
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@@
     (property "Reference" "U10" (id 0) (at 149.86 20.32 0))
     (property "Value" "TX4138" (id 1) (at 149.86 22.86 0))
-    (property "Footprint" "Package_SO:SOIC-8-1EP_3.9x4.9mm_P1.27mm_EP2.41x3.81mm_ThermalVias" (id 2) (at 151.13 36.83 0)
+    (property "Footprint" "Tales:SOIC-8-1EP_3.9x4.9mm_P1.27mm_EP2.29x3mm_ThermalVias" (id 2) (at 151.13 36.83 0)
       (effects (font (size 1.27 1.27)) hide)
     )
@@
       (effects (font (size 1.27 1.27)) (justify left))
     )
-    (property "Value" "12pF/50V/0603" (id 1) (at 107.95 68.58 0)
+    (property "Value" "22pF/50V/0603" (id 1) (at 107.95 68.58 0)
       (effects (font (size 1.27 1.27)) (justify left))
     )
@@
       (effects (font (size 1.27 1.27)) hide)
     )
-    (property "LCSC Part" "C38523" (id 6) (at 107.95 73.66 0)
+    (property "LCSC Part" "C1653" (id 6) (at 107.95 73.66 0)
       (effects (font (size 1.27 1.27)) (justify left))
     )
@@
       (effects (font (size 1.27 1.27)) hide)
     )
-    (property "Mfr PN" "CL10C120JB8NNNC" (id 8) (at 105.41 69.85 0)
+    (property "Mfr PN" "CL10C220JB8NNNC" (id 8) (at 105.41 69.85 0)
       (effects (font (size 1.27 1.27)) hide)
     )
@@
       (effects (font (size 1.27 1.27)) hide)
     )
-    (property "Vendor PN" "C38523" (id 11) (at 105.41 69.85 0)
+    (property "Vendor PN" "C1653" (id 11) (at 105.41 69.85 0)
       (effects (font (size 1.27 1.27)) hide)
     )
@@
       (effects (font (size 1.27 1.27)) (justify left))
     )
-    (property "Value" "300k/0,125W/0805" (id 1) (at 128.27 71.1199 0)
+    (property "Value" "100k/0,125W/0805" (id 1) (at 128.27 71.1199 0)
       (effects (font (size 1.27 1.27)) (justify left))
     )
@@
       (effects (font (size 1.27 1.27)) hide)
     )
-    (property "LCSC Part" "C17616" (id 6) (at 125.73 69.85 0)
+    (property "LCSC Part" "C149504" (id 6) (at 125.73 69.85 0)
       (effects (font (size 1.27 1.27)) hide)
     )
@@
       (effects (font (size 1.27 1.27)) hide)
     )
-    (property "Mfr PN" "0805W8F3003T5E" (id 8) (at 125.73 69.85 0)
+    (property "Mfr PN" "0805W8F1003T5E" (id 8) (at 125.73 69.85 0)
       (effects (font (size 1.27 1.27)) hide)
     )
@@
       (effects (font (size 1.27 1.27)) hide)
     )
-    (property "Vendor PN" "C17616" (id 11) (at 125.73 69.85 0)
+    (property "Vendor PN" "C149504" (id 11) (at 125.73 69.85 0)
       (effects (font (size 1.27 1.27)) hide)
     )
@@
       (effects (font (size 1.27 1.27)) (justify left))
     )
-    (property "Value" "10uF/16V/4x5,7" (id 1) (at 72.39 80.8481 0)
+    (property "Value" "10uF/16V/1206" (id 1) (at 72.39 80.8481 0)
       (effects (font (size 1.27 1.27)) (justify left))
     )
-    (property "Footprint" "Tales:CP_Elec_4x5.7" (id 2) (at 69.85 80.01 0)
+    (property "Footprint" "Tales:C_1206_3216Metric" (id 2) (at 69.85 80.01 0)
       (effects (font (size 1.27 1.27)) hide)
     )
@@
       (effects (font (size 1.27 1.27)) hide)
     )
-    (property "Mfr" "Lelon" (id 4) (at 69.85 80.01 0)
+    (property "Mfr" "Samsung" (id 4) (at 69.85 80.01 0)
       (effects (font (size 1.27 1.27)) hide)
     )
-    (property "Mfr PN" "VEU100M1CTR-0406" (id 5) (at 69.85 80.01 0)
+    (property "Mfr PN" "CL31A106KOHNNNE" (id 5) (at 69.85 80.01 0)
       (effects (font (size 1.27 1.27)) hide)
     )
@@
       (effects (font (size 1.27 1.27)) hide)
     )
-    (property "LCSC Part" "C249724" (id 7) (at 69.85 80.01 0)
+    (property "LCSC Part" "C1849" (id 7) (at 69.85 80.01 0)
       (effects (font (size 1.27 1.27)) hide)
     )
-    (property "Technology" "Electrolitic" (id 8) (at 69.85 80.01 0)
+    (property "Technology" "Ceramic" (id 8) (at 69.85 80.01 0)
       (effects (font (size 1.27 1.27)) hide)
     )
@@
       (effects (font (size 1.27 1.27)) hide)
     )
-    (property "Vendor PN" "C249724" (id 10) (at 69.85 80.01 0)
+    (property "Vendor PN" "C1849" (id 10) (at 69.85 80.01 0)
       (effects (font (size 1.27 1.27)) hide)
     )
-    (property "Case" "4x5,7" (id 11) (at 69.85 80.01 0)
+    (property "Case" "1206/3216" (id 11) (at 69.85 80.01 0)
       (effects (font (size 1.27 1.27)) hide)
     )
@@
       (effects (font (size 1.27 1.27)) (justify left))
     )
-    (property "Value" "57,6k/0,125W/0805" (id 1) (at 128.27 83.8199 0)
+    (property "Value" "22,1k/0,125W/0805" (id 1) (at 128.27 83.8199 0)
       (effects (font (size 1.27 1.27)) (justify left))
     )
@@
       (effects (font (size 1.27 1.27)) hide)
     )
-    (property "LCSC Part" "C17758" (id 6) (at 125.73 82.55 0)
+    (property "LCSC Part" "C17552" (id 6) (at 125.73 82.55 0)
       (effects (font (size 1.27 1.27)) hide)
     )
@@
       (effects (font (size 1.27 1.27)) hide)
     )
-    (property "Mfr PN" "0805W8F5762T5E" (id 8) (at 125.73 82.55 0)
+    (property "Mfr PN" "0805W8F2212T5E" (id 8) (at 125.73 82.55 0)
       (effects (font (size 1.27 1.27)) hide)
     )
@@
       (effects (font (size 1.27 1.27)) hide)
     )
-    (property "Vendor PN" "C17758" (id 11) (at 125.73 82.55 0)
+    (property "Vendor PN" "C17552" (id 11) (at 125.73 82.55 0)
       (effects (font (size 1.27 1.27)) hide)
     )
@@
       (effects (font (size 1.27 1.27)) (justify left))
     )
-    (property "Value" "10uF/16V/4x5,7" (id 1) (at 153.67 70.6881 0)
+    (property "Value" "10uF/16V/1206" (id 1) (at 153.67 70.6881 0)
       (effects (font (size 1.27 1.27)) (justify left))
     )
-    (property "Footprint" "Tales:CP_Elec_4x5.7" (id 2) (at 151.13 69.85 0)
+    (property "Footprint" "Tales:C_1206_3216Metric" (id 2) (at 151.13 69.85 0)
       (effects (font (size 1.27 1.27)) hide)
     )
@@
       (effects (font (size 1.27 1.27)) hide)
     )
-    (property "Mfr" "Lelon" (id 4) (at 151.13 69.85 0)
+    (property "Mfr" "Samsung" (id 4) (at 151.13 69.85 0)
       (effects (font (size 1.27 1.27)) hide)
     )
-    (property "Mfr PN" "VEU100M1CTR-0406" (id 5) (at 151.13 69.85 0)
+    (property "Mfr PN" "CL31A106KOHNNNE" (id 5) (at 151.13 69.85 0)
       (effects (font (size 1.27 1.27)) hide)
     )
@@
       (effects (font (size 1.27 1.27)) hide)
     )
-    (property "LCSC Part" "C249724" (id 7) (at 151.13 69.85 0)
+    (property "LCSC Part" "C1849" (id 7) (at 151.13 69.85 0)
       (effects (font (size 1.27 1.27)) hide)
     )
-    (property "Technology" "Electrolitic" (id 8) (at 151.13 69.85 0)
+    (property "Technology" "Ceramic" (id 8) (at 151.13 69.85 0)
       (effects (font (size 1.27 1.27)) hide)
     )
@@
       (effects (font (size 1.27 1.27)) hide)
     )
-    (property "Vendor PN" "C249724" (id 10) (at 151.13 69.85 0)
+    (property "Vendor PN" "C1849" (id 10) (at 151.13 69.85 0)
       (effects (font (size 1.27 1.27)) hide)
     )
-    (property "Case" "4x5,7" (id 11) (at 151.13 69.85 0)
+    (property "Case" "1206/3216" (id 11) (at 151.13 69.85 0)
       (effects (font (size 1.27 1.27)) hide)
     )
@@
     (property "Reference" "U1" (id 0) (at 81.28 53.34 0))
     (property "Value" "SY8089A1AAC" (id 1) (at 81.28 55.88 0))
-    (property "Footprint" "Package_TO_SOT_SMD:TSOT-23-5" (id 2) (at 81.28 67.31 0)
+    (property "Footprint" "Tales:TSOT-23-5" (id 2) (at 81.28 67.31 0)
       (effects (font (size 1.27 1.27)) hide)
     )
@@
     )
     (path "/9ce2d269-207e-428e-8bde-8f81e24185ac"
-      (reference "C1") (unit 1) (value "10uF/16V/4x5,7") (footprint "Tales:CP_Elec_4x5.7")
+      (reference "C1") (unit 1) (value "10uF/16V/1206") (footprint "Tales:C_1206_3216Metric")
     )
     (path "/00000000-0000-0000-0000-000062418b8f"
@@
     )
     (path "/180c977c-9b8e-42f5-b6a5-5ecbfddc8a10"
-      (reference "C12") (unit 1) (value "12pF/50V/0603") (footprint "Tales:C_0603_1608Metric")
+      (reference "C12") (unit 1) (value "22pF/50V/0603") (footprint "Tales:C_0603_1608Metric")
     )
     (path "/ea9b47d9-fa0f-4b54-91b9-ea103ad3c576"
-      (reference "C13") (unit 1) (value "10uF/16V/4x5,7") (footprint "Tales:CP_Elec_4x5.7")
+      (reference "C13") (unit 1) (value "10uF/16V/1206") (footprint "Tales:C_1206_3216Metric")
     )
     (path "/37817d52-9c5e-4e0a-8d56-12eacc35b998"
@@
     )
     (path "/4d7fb05d-70f8-441c-acfd-65f8f8e18048"
-      (reference "R10") (unit 1) (value "300k/0,125W/0805") (footprint "Tales:R_0805_2012Metric")
+      (reference "R10") (unit 1) (value "100k/0,125W/0805") (footprint "Tales:R_0805_2012Metric")
     )
     (path "/e5155ad6-8e84-4d81-b834-9be26b20abe3"
-      (reference "R11") (unit 1) (value "57,6k/0,125W/0805") (footprint "Tales:R_0805_2012Metric")
+      (reference "R11") (unit 1) (value "22,1k/0,125W/0805") (footprint "Tales:R_0805_2012Metric")
     )
     (path "/00000000-0000-0000-0000-000062418b42"
@@
     )
     (path "/f980e0df-dacc-4bad-af81-dac62143b6ee"
-      (reference "U1") (unit 1) (value "SY8089A1AAC") (footprint "Package_TO_SOT_SMD:TSOT-23-5")
+      (reference "U1") (unit 1) (value "SY8089A1AAC") (footprint "Tales:TSOT-23-5")
     )
     (path "/e41c8ba8-d546-4f8b-b36a-c7995cebe79c"
@@
     )
     (path "/177a016e-6798-4372-b14c-8df883d58d2b"
-      (reference "U10") (unit 1) (value "TX4138") (footprint "Package_SO:SOIC-8-1EP_3.9x4.9mm_P1.27mm_EP2.41x3.81mm_ThermalVias")
+      (reference "U10") (unit 1) (value "TX4138") (footprint "Tales:SOIC-8-1EP_3.9x4.9mm_P1.27mm_EP2.29x3mm_ThermalVias")
     )
     (path "/00000000-0000-0000-0000-000060761483"

Commit message: Development
Parts:
- C1, C13: LCSC Part C1849 -> (none); LCSC Part # (none) -> C1849
- C10, C3, C4, C5, C6, C7, C8, C9: LCSC Part C1739 -> (none); LCSC Part # (none) -> C1739
- C11, C14: LCSC Part C49678 -> (none); LCSC Part # (none) -> C49678
- C12: LCSC Part C1653 -> (none); LCSC Part # (none) -> C1653
- C15: LCSC Part C38523 -> (none); LCSC Part # (none) -> C38523
- C16: LCSC Part C249930 -> (none); LCSC Part # (none) -> C249930
- C2: LCSC Part C263963 -> (none); LCSC Part # (none) -> C263963
- D1: LCSC Part C64898 -> (none); LCSC Part # (none) -> C64898
- D10: LCSC Part C65010 -> (none); LCSC Part # (none) -> C65010
- D11, D12, D13, D14, D19, D20, D21, D22: LCSC Part C72041 -> (none); LCSC Part # (none) -> C72041
- D15, D16, D17, D18, D24, D25, D26, D27: LCSC Part C81598 -> (none); LCSC Part # (none) -> C81598
- D2, D3, D4, D5, D6, D7, D8, D9: LCSC Part C109072 -> (none); LCSC Part # (none) -> C109072
- D23, D28, D29: LCSC Part C72043 -> (none); LCSC Part # (none) -> C72043
- J1: JLCPCB BOM (none) -> 0; Mfr (none) -> Metaltex; Mfr PN (none) -> BR902V; Vendor (none) -> Eletropeças; Vendor PN (none) -> 29273
- J10: value OUT1 -> OUT8
- J4: value OUT1 -> OUT2
- J5: value OUT1 -> OUT3
- J6: value OUT1 -> OUT4
- J7: value OUT1 -> OUT5
- J8: value OUT1 -> OUT6
- J9: value OUT1 -> OUT7
- L1: LCSC Part C370424 -> (none); LCSC Part # (none) -> C370424
- L2: LCSC Part C127788 -> (none); LCSC Part # (none) -> C127788
- Q1, Q2, Q3, Q4, Q5, Q6, Q7, Q8: LCSC Part C8512 -> (none); LCSC Part # (none) -> C8512
- R1, R2, R3, R4, R5, R6, R7, R8: LCSC Part C17379 -> (none); LCSC Part # (none) -> C17379
- R10: LCSC Part C149504 -> (none); LCSC Part # (none) -> C149504
- R11: LCSC Part C17552 -> (none); LCSC Part # (none) -> C17552
- R12, R13, R14, R15, R16, R17, R18, R19: LCSC Part C26010 -> (none); LCSC Part # (none) -> C26010
- R20: LCSC Part C17724 -> (none); LCSC Part # (none) -> C17724
- R21, R23, R25, R27, R35, R36, R38, R40, R42: LCSC Part C17673 -> (none); LCSC Part # (none) -> C17673
- R22, R24, R26, R28, R37, R39, R41, R43: LCSC Part C17414 -> (none); LCSC Part # (none) -> C17414
- R29: LCSC Part C17616 -> (none); LCSC Part # (none) -> C17616
- R30: LCSC Part C17758 -> (none); LCSC Part # (none) -> C17758
- R31, R32, R33, R34, R45, R46, R47, R48: LCSC Part C17513 -> (none); LCSC Part # (none) -> C17513
- R44: LCSC Part C4382 -> (none); LCSC Part # (none) -> C4382
- R49: LCSC Part C17837 -> (none); LCSC Part # (none) -> C17837
- R50: LCSC Part C17630 -> (none); LCSC Part # (none) -> C17630
- R9: LCSC Part C247605 -> (none); LCSC Part # (none) -> C247605
- U1: LCSC Part C479074 -> (none); LCSC Part # (none) -> C479074
- U10: LCSC Part C329267 -> (none); LCSC Part # (none) -> C329267
- U2, U3, U4, U5, U6, U7, U8, U9: LCSC Part C109227 -> (none); LCSC Part # (none) -> C109227
