File: V1/ESP-relay-8ch-V1.kicad_sch (KiCad schematic)
At the start: 142 parts, among them J1 +24VDC, J10 OUT8, J2 INPUTS, J3 OUT1, J4 OUT2, J5 OUT3, J6 OUT4, J7 OUT5, J8 OUT6, J9 OUT7, K1 G5PZ-1A, K2 G5PZ-1A, K3 G5PZ-1A, K4 G5PZ-1A, K5 G5PZ-1A, K6 G5PZ-1A, K7 G5PZ-1A, K8 G5PZ-1A, Q1 MMBT2222A/SOT-23-3, Q2 MMBT2222A/SOT-23-3, Q3 MMBT2222A/SOT-23-3, Q4 MMBT2222A/SOT-23-3, Q5 MMBT2222A/SOT-23-3, Q6 MMBT2222A/SOT-23-3, Q7 MMBT2222A/SOT-23-3, Q8 MMBT2222A/SOT-23-3, U1 SY8089A1AAC, U10 TX4138, U11 Olimex_ESP32-POE, U2 LTV-817S, U3 LTV-817S, U4 LTV-817S, U5 LTV-817S, U6 LTV-817S, U7 LTV-817S, U8 LTV-817S, U9 LTV-817S

Commit message: SCH tweaks
Parts:
- C1, C13: Technology Ceramic -> Ceramic X5R
Changed lines of the file:
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@@
   (symbol (lib_id "Tales:Olimex_ESP32-POE") (at 289.56 46.99 0) (unit 1)
     (in_bom yes) (on_board yes)
-    (property "Reference" "U11" (id 0) (at 312.42 24.13 0))
-    (property "Value" "Olimex_ESP32-POE" (id 1) (at 312.42 26.67 0))
+    (property "Reference" "U11" (id 0) (at 303.53 24.13 0))
+    (property "Value" "Olimex_ESP32-POE" (id 1) (at 304.8 26.67 0))
     (property "Footprint" "Tales:Olimex_ESP32-POE" (id 2) (at 289.56 76.2 0)
       (effects (font (size 1.27 1.27)) hide)
@@
   (symbol (lib_id "Device:L") (at 97.79 63.5 90) (unit 1)
     (in_bom yes) (on_board yes)
-    (property "Reference" "L1" (id 0) (at 97.79 66.04 90))
-    (property "Value" "2,2uH" (id 1) (at 97.79 68.58 90))
+    (property "Reference" "L1" (id 0) (at 97.79 55.88 90))
+    (property "Value" "2,2uH" (id 1) (at 97.79 58.42 90))
     (property "Footprint" "Tales:L_3x3_H1.5" (id 2) (at 97.79 63.5 0)
       (effects (font (size 1.27 1.27)) hide)
@@
       (effects (font (size 1.27 1.27)) hide)
     )
-    (property "LCSC Part #" "C370424" (id 6) (at 97.79 71.12 90))
+    (property "LCSC Part #" "C370424" (id 6) (at 97.79 60.96 90))
     (property "Mfr" "Sunlord" (id 7) (at 97.79 63.5 0)
       (effects (font (size 1.27 1.27)) hide)
@@
   )
   (symbol (lib_id "Device:C_Polarized_Small_US") (at 234.95 46.99 0) (unit 1)
-    (in_bom yes) (on_board yes) (fields_autoplaced)
-    (property "Reference" "C16" (id 0) (at 237.49 45.2881 0)
+    (in_bom yes) (on_board yes)
+    (property "Reference" "C16" (id 0) (at 237.49 44.45 0)
       (effects (font (size 1.27 1.27)) (justify left))
     )
-    (property "Value" "470uF/16V/10x10" (id 1) (at 237.49 47.8281 0)
+    (property "Value" "470uF/16V/10x10" (id 1) (at 237.49 46.99 0)
       (effects (font (size 1.27 1.27)) (justify left))
     )
@@
       (effects (font (size 1.27 1.27)) hide)
     )
-    (property "LCSC Part #" "C249930" (id 7) (at 234.95 46.99 0)
-      (effects (font (size 1.27 1.27)) hide)
+    (property "LCSC Part #" "C249930" (id 7) (at 237.49 52.07 0)
+      (effects (font (size 1.27 1.27)) (justify left))
     )
-    (property "Technology" "Electrolitic" (id 8) (at 234.95 46.99 0)
-      (effects (font (size 1.27 1.27)) hide)
+    (property "Technology" "Electrolitic" (id 8) (at 237.49 49.53 0)
+      (effects (font (size 1.27 1.27)) (justify left))
     )
     (property "Vendor" "JLCPCB" (id 9) (at 234.95 46.99 0)
@@
   )
   (symbol (lib_id "Device:R_US") (at 125.73 69.85 0) (unit 1)
-    (in_bom yes) (on_board yes) (fields_autoplaced)
-    (property "Reference" "R10" (id 0) (at 128.27 68.5799 0)
+    (in_bom yes) (on_board yes)
+    (property "Reference" "R10" (id 0) (at 128.27 68.58 0)
       (effects (font (size 1.27 1.27)) (justify left))
     )
-    (property "Value" "100k/0,125W/0805" (id 1) (at 128.27 71.1199 0)
+    (property "Value" "100k/0,125W/0805" (id 1) (at 128.27 71.12 0)
       (effects (font (size 1.27 1.27)) (justify left))
     )
@@
       (effects (font (size 1.27 1.27)) hide)
     )
-    (property "LCSC Part #" "C149504" (id 6) (at 125.73 69.85 0)
-      (effects (font (size 1.27 1.27)) hide)
+    (property "LCSC Part #" "C149504" (id 6) (at 128.27 73.66 0)
+      (effects (font (size 1.27 1.27)) (justify left))
     )
     (property "Mfr" "Uniroyal" (id 7) (at 125.73 69.85 0)
@@
   )
   (symbol (lib_id "Device:C_Polarized_Small_US") (at 69.85 80.01 0) (unit 1)
-    (in_bom yes) (on_board yes) (fields_autoplaced)
-    (property "Reference" "C1" (id 0) (at 72.39 78.3081 0)
+    (in_bom yes) (on_board yes)
+    (property "Reference" "C1" (id 0) (at 72.39 78.105 0)
       (effects (font (size 1.27 1.27)) (justify left))
     )
-    (property "Value" "10uF/16V/1206" (id 1) (at 72.39 80.8481 0)
+    (property "Value" "10uF/16V/1206" (id 1) (at 72.39 80.645 0)
       (effects (font (size 1.27 1.27)) (justify left))
     )
@@
       (effects (font (size 1.27 1.27)) hide)
     )
-    (property "LCSC Part #" "C1849" (id 7) (at 69.85 80.01 0)
-      (effects (font (size 1.27 1.27)) hide)
+    (property "LCSC Part #" "C1849" (id 7) (at 72.39 85.725 0)
+      (effects (font (size 1.27 1.27)) (justify left))
     )
-    (property "Technology" "Ceramic" (id 8) (at 69.85 80.01 0)
-      (effects (font (size 1.27 1.27)) hide)
+    (property "Technology" "Ceramic X5R" (id 8) (at 72.39 83.185 0)
+      (effects (font (size 1.27 1.27)) (justify left))
     )
     (property "Vendor" "JLCPCB" (id 9) (at 69.85 80.01 0)
@@
   )
   (symbol (lib_id "Device:R_US") (at 210.82 46.99 0) (unit 1)
-    (in_bom yes) (on_board yes) (fields_autoplaced)
-    (property "Reference" "R29" (id 0) (at 213.36 45.7199 0)
+    (in_bom yes) (on_board yes)
+    (property "Reference" "R29" (id 0) (at 213.36 44.45 0)
       (effects (font (size 1.27 1.27)) (justify left))
     )
-    (property "Value" "300k/0,125W/0805" (id 1) (at 213.36 48.2599 0)
+    (property "Value" "300k/0,125W/0805" (id 1) (at 213.36 46.99 0)
       (effects (font (size 1.27 1.27)) (justify left))
     )
@@
       (effects (font (size 1.27 1.27)) hide)
     )
-    (property "LCSC Part #" "C17616" (id 6) (at 210.82 46.99 0)
-      (effects (font (size 1.27 1.27)) hide)
+    (property "LCSC Part #" "C17616" (id 6) (at 213.36 49.53 0)
+      (effects (font (size 1.27 1.27)) (justify left))
     )
     (property "Mfr" "Uniroyal" (id 7) (at 210.82 46.99 0)
@@
   )
   (symbol (lib_id "Device:R_US") (at 210.82 60.96 0) (unit 1)
-    (in_bom yes) (on_board yes) (fields_autoplaced)
-    (property "Reference" "R30" (id 0) (at 213.36 59.6899 0)
+    (in_bom yes) (on_board yes)
+    (property "Reference" "R30" (id 0) (at 213.36 58.42 0)
       (effects (font (size 1.27 1.27)) (justify left))
     )
-    (property "Value" "57,6k/0,125W/0805" (id 1) (at 213.36 62.2299 0)
+    (property "Value" "57,6k/0,125W/0805" (id 1) (at 213.36 60.96 0)
       (effects (font (size 1.27 1.27)) (justify left))
     )
@@
       (effects (font (size 1.27 1.27)) hide)
     )
-    (property "LCSC Part #" "C17758" (id 6) (at 210.82 60.96 0)
-      (effects (font (size 1.27 1.27)) hide)
+    (property "LCSC Part #" "C17758" (id 6) (at 213.36 63.5 0)
+      (effects (font (size 1.27 1.27)) (justify left))
     )
     (property "Mfr" "Uniroyal" (id 7) (at 210.82 60.96 0)
@@
   (symbol (lib_id "Device:D_Schottky") (at 167.64 45.72 270) (unit 1)
     (in_bom yes) (on_board yes)
-    (property "Reference" "D10" (id 0) (at 170.18 44.1324 90)
+    (property "Reference" "D10" (id 0) (at 170.18 43.18 90)
       (effects (font (size 1.27 1.27)) (justify left))
     )
-    (property "Value" "SS510" (id 1) (at 170.18 46.6724 90)
+    (property "Value" "SS510" (id 1) (at 170.18 45.72 90)
       (effects (font (size 1.27 1.27)) (justify left))
     )
@@
       (effects (font (size 1.27 1.27)) hide)
     )
-    (property "LCSC Part #" "C65010" (id 6) (at 170.18 49.53 90)
+    (property "LCSC Part #" "C65010" (id 6) (at 170.18 48.26 90)
       (effects (font (size 1.27 1.27)) (justify left))
     )
@@
   )
   (symbol (lib_id "Device:R_US") (at 125.73 82.55 0) (unit 1)
-    (in_bom yes) (on_board yes) (fields_autoplaced)
-    (property "Reference" "R11" (id 0) (at 128.27 81.2799 0)
+    (in_bom yes) (on_board yes)
+    (property "Reference" "R11" (id 0) (at 128.27 81.28 0)
       (effects (font (size 1.27 1.27)) (justify left))
     )
-    (property "Value" "22,1k/0,125W/0805" (id 1) (at 128.27 83.8199 0)
+    (property "Value" "22,1k/0,125W/0805" (id 1) (at 128.27 83.82 0)
       (effects (font (size 1.27 1.27)) (justify left))
     )
@@
       (effects (font (size 1.27 1.27)) hide)
     )
-    (property "LCSC Part #" "C17552" (id 6) (at 125.73 82.55 0)
-      (effects (font (size 1.27 1.27)) hide)
+    (property "LCSC Part #" "C17552" (id 6) (at 128.27 86.36 0)
+      (effects (font (size 1.27 1.27)) (justify left))
     )
     (property "Mfr" "Uniroyal" (id 7) (at 125.73 82.55 0)
@@
   )
   (symbol (lib_id "Device:C_Polarized_Small_US") (at 151.13 69.85 0) (unit 1)
-    (in_bom yes) (on_board yes) (fields_autoplaced)
-    (property "Reference" "C13" (id 0) (at 153.67 68.1481 0)
+    (in_bom yes) (on_board yes)
+    (property "Reference" "C13" (id 0) (at 153.67 66.04 0)
       (effects (font (size 1.27 1.27)) (justify left))
     )
-    (property "Value" "10uF/16V/1206" (id 1) (at 153.67 70.6881 0)
+    (property "Value" "10uF/16V/1206" (id 1) (at 153.67 68.58 0)
       (effects (font (size 1.27 1.27)) (justify left))
     )
@@
       (effects (font (size 1.27 1.27)) hide)
     )
-    (property "LCSC Part #" "C1849" (id 7) (at 151.13 69.85 0)
-      (effects (font (size 1.27 1.27)) hide)
+    (property "LCSC Part #" "C1849" (id 7) (at 153.67 73.66 0)
+      (effects (font (size 1.27 1.27)) (justify left))
     )
-    (property "Technology" "Ceramic" (id 8) (at 151.13 69.85 0)
-      (effects (font (size 1.27 1.27)) hide)
+    (property "Technology" "Ceramic X5R" (id 8) (at 153.67 71.12 0)
+      (effects (font (size 1.27 1.27)) (justify left))
     )
     (property "Vendor" "JLCPCB" (id 9) (at 151.13 69.85 0)
