File: V1/ESP-relay-8ch-V1.kicad_sch (KiCad schematic)
At the start: 143 parts, among them J1 +24VDC, J10 OUT8, J2 INPUTS, J3 OUT1, J4 OUT2, J5 OUT3, J6 OUT4, J7 OUT5, J8 OUT6, J9 OUT7, K1 G5PZ-1A, K2 G5PZ-1A, K3 G5PZ-1A, K4 G5PZ-1A, K5 G5PZ-1A, K6 G5PZ-1A, K7 G5PZ-1A, K8 G5PZ-1A, Q1 MMBT2222A/SOT-23-3, Q2 MMBT2222A/SOT-23-3, Q3 MMBT2222A/SOT-23-3, Q4 MMBT2222A/SOT-23-3, Q5 MMBT2222A/SOT-23-3, Q6 MMBT2222A/SOT-23-3, Q7 MMBT2222A/SOT-23-3, Q8 MMBT2222A/SOT-23-3, U1 SY8089A1AAC, U10 TX4138, U11 Olimex_ESP32-POE, U2 LTV-817S, U3 LTV-817S, U4 LTV-817S, U5 LTV-817S, U6 LTV-817S, U7 LTV-817S, U8 LTV-817S, U9 LTV-817S

Commit message: PCB updates
Parts:
- removed D23, D28, D29: GREEN/0603, Tales:LED_0603_1608Metric, symbol Device:LED
- added D3, D4, D5: BLUE/0603, Tales:LED_0603_1608Metric, symbol Device:LED
- renumbered C2 to C1, C4 to C10, C5 to C11, C6 to C12, C7 to C13, C8 to C14, C9 to C15, C10 to C16, C11 to C2, C14 to C3, C15 to C4, C16 to C5, C1 to C6, C12 to C7, C13 to C8, C3 to C9, D6 to D10, D7 to D11, D8 to D12, D9 to D13, D11 to D14, D12 to D16, D16 to D17, D13 to D18, D17 to D19, D10 to D2, D14 to D20, D18 to D21, D19 to D22, D24 to D23, D20 to D24, D21 to D26, D26 to D27, D22 to D28, D27 to D29, D2 to D6, D3 to D7, D4 to D8, D5 to D9, R9 to R1, R11 to R10, R1 to R11, R2 to R13, R13 to R14, R3 to R15, R14 to R16, R4 to R17, R15 to R18, R5 to R19, R20 to R2, R16 to R20, R6 to R21, R17 to R22, R7 to R23, R18 to R24, R8 to R25, R19 to R26, R21 to R27, R22 to R28, R31 to R29, R29 to R3, R23 to R30, R24 to R31, R25 to R33, R26 to R34, R33 to R35, R27 to R36, R28 to R37, R34 to R38, R36 to R39, R30 to R4, R37 to R40, R45 to R41, R38 to R42, R39 to R43, R46 to R44, R40 to R45, R41 to R46, R42 to R48, R43 to R49, R35 to R5, R48 to R50, R44 to R6, R49 to R7, R50 to R8, R10 to R9, U10 to U1, U8 to U10, U9 to U11, U1 to U2, U11 to U3, U2 to U4, U3 to U5, U4 to U6, U5 to U7, U6 to U8, U7 to U9
Connections:
- net GNDREF: now also D3.1 (K), D4.1 (K), D5.1 (K)
- net at R6.2: now also D3.2 (A)
- net at R7.2: now also D4.2 (A)
- net at R8.2: now also D5.2 (A)

Commit message: JLCPCB part update
Parts:
- D10, D11, D12, D13, D6, D7, D8, D9: LCSC Part # C109072 -> C8067; Mfr PN ZMM5239B -> ZMM9V1-M; Vendor PN C109072 -> C8067
Changed lines of the file:
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@@
       (effects (font (size 1.27 1.27)) hide)
     )
-    (property "Mfr PN" "ZMM5239B" (id 6) (at 115.57 110.49 0)
+    (property "Mfr PN" "ZMM9V1-M" (id 6) (at 115.57 110.49 0)
       (effects (font (size 1.27 1.27)) hide)
     )
@@
       (effects (font (size 1.27 1.27)) hide)
     )
-    (property "Vendor PN" "C109072" (id 9) (at 115.57 110.49 0)
+    (property "Vendor PN" "C8067" (id 9) (at 115.57 110.49 0)
       (effects (font (size 1.27 1.27)) hide)
     )
@@
       (effects (font (size 1.27 1.27)) hide)
     )
-    (property "LCSC Part #" "C109072" (id 11) (at 115.57 107.95 0))
+    (property "LCSC Part #" "C8067" (id 11) (at 115.57 107.95 0))
     (pin "1")
     (pin "2")
@@
       (effects (font (size 1.27 1.27)) hide)
     )
-    (property "Mfr PN" "ZMM5239B" (id 6) (at 115.57 132.08 0)
+    (property "Mfr PN" "ZMM9V1-M" (id 6) (at 115.57 132.08 0)
       (effects (font (size 1.27 1.27)) hide)
     )
@@
       (effects (font (size 1.27 1.27)) hide)
     )
-    (property "Vendor PN" "C109072" (id 9) (at 115.57 132.08 0)
+    (property "Vendor PN" "C8067" (id 9) (at 115.57 132.08 0)
       (effects (font (size 1.27 1.27)) hide)
     )
@@
       (effects (font (size 1.27 1.27)) hide)
     )
-    (property "LCSC Part #" "C109072" (id 11) (at 115.57 129.54 0))
+    (property "LCSC Part #" "C8067" (id 11) (at 115.57 129.54 0))
     (pin "1")
     (pin "2")
@@
       (effects (font (size 1.27 1.27)) hide)
     )
-    (property "Mfr PN" "ZMM5239B" (id 6) (at 115.57 153.67 0)
+    (property "Mfr PN" "ZMM9V1-M" (id 6) (at 115.57 153.67 0)
       (effects (font (size 1.27 1.27)) hide)
     )
@@
       (effects (font (size 1.27 1.27)) hide)
     )
-    (property "Vendor PN" "C109072" (id 9) (at 115.57 153.67 0)
+    (property "Vendor PN" "C8067" (id 9) (at 115.57 153.67 0)
       (effects (font (size 1.27 1.27)) hide)
     )
@@
       (effects (font (size 1.27 1.27)) hide)
     )
-    (property "LCSC Part #" "C109072" (id 11) (at 115.57 151.13 0))
+    (property "LCSC Part #" "C8067" (id 11) (at 115.57 151.13 0))
     (pin "1")
     (pin "2")
@@
       (effects (font (size 1.27 1.27)) hide)
     )
-    (property "Mfr PN" "ZMM5239B" (id 6) (at 115.57 175.26 0)
+    (property "Mfr PN" "ZMM9V1-M" (id 6) (at 115.57 175.26 0)
       (effects (font (size 1.27 1.27)) hide)
     )
@@
       (effects (font (size 1.27 1.27)) hide)
     )
-    (property "Vendor PN" "C109072" (id 9) (at 115.57 175.26 0)
+    (property "Vendor PN" "C8067" (id 9) (at 115.57 175.26 0)
       (effects (font (size 1.27 1.27)) hide)
     )
@@
       (effects (font (size 1.27 1.27)) hide)
     )
-    (property "LCSC Part #" "C109072" (id 11) (at 115.57 172.72 0))
+    (property "LCSC Part #" "C8067" (id 11) (at 115.57 172.72 0))
     (pin "1")
     (pin "2")
@@
       (effects (font (size 1.27 1.27)) hide)
     )
-    (property "Mfr PN" "ZMM5239B" (id 6) (at 115.57 196.85 0)
+    (property "Mfr PN" "ZMM9V1-M" (id 6) (at 115.57 196.85 0)
       (effects (font (size 1.27 1.27)) hide)
     )
@@
       (effects (font (size 1.27 1.27)) hide)
     )
-    (property "Vendor PN" "C109072" (id 9) (at 115.57 196.85 0)
+    (property "Vendor PN" "C8067" (id 9) (at 115.57 196.85 0)
       (effects (font (size 1.27 1.27)) hide)
     )
@@
       (effects (font (size 1.27 1.27)) hide)
     )
-    (property "LCSC Part #" "C109072" (id 11) (at 115.57 194.31 0))
+    (property "LCSC Part #" "C8067" (id 11) (at 115.57 194.31 0))
     (pin "1")
     (pin "2")
@@
       (effects (font (size 1.27 1.27)) hide)
     )
-    (property "Mfr PN" "ZMM5239B" (id 6) (at 115.57 218.44 0)
+    (property "Mfr PN" "ZMM9V1-M" (id 6) (at 115.57 218.44 0)
       (effects (font (size 1.27 1.27)) hide)
     )
@@
       (effects (font (size 1.27 1.27)) hide)
     )
-    (property "Vendor PN" "C109072" (id 9) (at 115.57 218.44 0)
+    (property "Vendor PN" "C8067" (id 9) (at 115.57 218.44 0)
       (effects (font (size 1.27 1.27)) hide)
     )
@@
       (effects (font (size 1.27 1.27)) hide)
     )
-    (property "LCSC Part #" "C109072" (id 11) (at 115.57 215.9 0))
+    (property "LCSC Part #" "C8067" (id 11) (at 115.57 215.9 0))
     (pin "1")
     (pin "2")
@@
       (effects (font (size 1.27 1.27)) hide)
     )
-    (property "Mfr PN" "ZMM5239B" (id 6) (at 115.57 261.62 0)
+    (property "Mfr PN" "ZMM9V1-M" (id 6) (at 115.57 261.62 0)
       (effects (font (size 1.27 1.27)) hide)
     )
@@
       (effects (font (size 1.27 1.27)) hide)
     )
-    (property "Vendor PN" "C109072" (id 9) (at 115.57 261.62 0)
+    (property "Vendor PN" "C8067" (id 9) (at 115.57 261.62 0)
       (effects (font (size 1.27 1.27)) hide)
     )
@@
       (effects (font (size 1.27 1.27)) hide)
     )
-    (property "LCSC Part #" "C109072" (id 11) (at 115.57 259.08 0))
+    (property "LCSC Part #" "C8067" (id 11) (at 115.57 259.08 0))
     (pin "1")
     (pin "2")
@@
       (effects (font (size 1.27 1.27)) hide)
     )
-    (property "Mfr PN" "ZMM5239B" (id 6) (at 115.57 240.03 0)
+    (property "Mfr PN" "ZMM9V1-M" (id 6) (at 115.57 240.03 0)
       (effects (font (size 1.27 1.27)) hide)
     )
@@
       (effects (font (size 1.27 1.27)) hide)
     )
-    (property "Vendor PN" "C109072" (id 9) (at 115.57 240.03 0)
+    (property "Vendor PN" "C8067" (id 9) (at 115.57 240.03 0)
       (effects (font (size 1.27 1.27)) hide)
     )
@@
       (effects (font (size 1.27 1.27)) hide)
     )
-    (property "LCSC Part #" "C109072" (id 11) (at 115.57 237.49 0))
+    (property "LCSC Part #" "C8067" (id 11) (at 115.57 237.49 0))
     (pin "1")
     (pin "2")
