File: V1/ESP-relay-8ch-V1.kicad_sch (KiCad schematic)
At the start: 143 parts, among them J1 +24VDC, J10 OUT8, J2 INPUTS, J3 OUT1, J4 OUT2, J5 OUT3, J6 OUT4, J7 OUT5, J8 OUT6, J9 OUT7, K1 G5PZ-1A, K2 G5PZ-1A, K3 G5PZ-1A, K4 G5PZ-1A, K5 G5PZ-1A, K6 G5PZ-1A, K7 G5PZ-1A, K8 G5PZ-1A, Q1 MMBT2222A/SOT-23-3, Q2 MMBT2222A/SOT-23-3, Q3 MMBT2222A/SOT-23-3, Q4 MMBT2222A/SOT-23-3, Q5 MMBT2222A/SOT-23-3, Q6 MMBT2222A/SOT-23-3, Q7 MMBT2222A/SOT-23-3, Q8 MMBT2222A/SOT-23-3, U1 TX4138, U10 LTV-817S, U11 LTV-817S, U2 SY8089A1AAC, U3 Olimex_ESP32-POE, U4 LTV-817S, U5 LTV-817S, U6 LTV-817S, U7 LTV-817S, U8 LTV-817S, U9 LTV-817S

Commit message: Design optimization
Parts:
- removed LOGO1: Logo_Open_Hardware_Large, Symbol:OSHW-Logo2_14.6x12mm_SilkScreen, symbol Graphic:Logo_Open_Hardware_Large
Other:
- note removed: "OPEN HARDWARE"
Changed lines of the file:
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@@
     (stroke (width 0) (type default))
   )
-  (text "OPEN HARDWARE" (at 16.51 279.4 0)
-    (effects (font (size 3 3)) (justify left bottom))
-  )
   (global_label "OUT2" (shape input) (at 313.69 46.99 0) (fields_autoplaced)
     (effects (font (size 1.27 1.27)) (justify left))
@@
         )
       )
-    )
-  )
-  (symbol (lib_id "Graphic:Logo_Open_Hardware_Large") (at 35.56 264.16 0) (unit 1)
-    (in_bom yes) (on_board yes) (dnp no) (fields_autoplaced)
-    (property "Reference" "LOGO1" (at 35.56 251.46 0)
-      (effects (font (size 1.27 1.27)) hide)
-    )
-    (property "Value" "Logo_Open_Hardware_Large" (at 35.56 274.32 0)
-      (effects (font (size 1.27 1.27)) hide)
-    )
-    (property "Footprint" "Symbol:OSHW-Logo2_14.6x12mm_SilkScreen" (at 35.56 264.16 0)
-      (effects (font (size 1.27 1.27)) hide)
-    )
-    (property "Datasheet" "~" (at 35.56 264.16 0)
-      (effects (font (size 1.27 1.27)) hide)
-    )
-    (instances
-      (project "ESP-relay-8ch-V1"
-        (path "/2bc5a21a-1d79-419d-a592-6852cc07b00a"
-          (reference "LOGO1") (unit 1)
-        )
-      )
