File: V2/ESP-relay-8ch-V2.kicad_pcb (KiCad board)
At the start: 2 copper layers, 198 x 67.8 mm, 143 parts, among them J1 +24VDC, J10 OUT8, J2 INPUTS, J3 OUT1, J4 OUT2, J5 OUT3, J6 OUT4, J7 OUT5, J8 OUT6, J9 OUT7, K1 G5PZ-1A, K2 G5PZ-1A, K3 G5PZ-1A, K4 G5PZ-1A, K5 G5PZ-1A, K6 G5PZ-1A, K7 G5PZ-1A, K8 G5PZ-1A, Q1 MMBT2222A/SOT-23-3, Q2 MMBT2222A/SOT-23-3, Q3 MMBT2222A/SOT-23-3, Q4 MMBT2222A/SOT-23-3, Q5 MMBT2222A/SOT-23-3, Q6 MMBT2222A/SOT-23-3, Q7 MMBT2222A/SOT-23-3, Q8 MMBT2222A/SOT-23-3, U1 SY8089A1AAC, U10 TX4138, U11 Olimex_ESP32-POE, U2 LTV-817S, U3 LTV-817S, U4 LTV-817S, U5 LTV-817S, U6 LTV-817S, U7 LTV-817S, U8 LTV-817S, U9 LTV-817S

Commit message: Dev
Parts:
- removed LOGO1: Logo_Open_Hardware_Large, Symbol:OSHW-Logo2_14.6x12mm_SilkScreen
- added J11: RJ45_LED, Connector_RJ:RJ45_Amphenol_RJHSE538X, F.Cu at (144.8, 123.2)
- added U12: LAN8710A, Package_DFN_QFN:QFN-32-1EP_5x5mm_P0.5mm_EP3.3x3.3mm_ThermalVias, F.Cu at (143.4, 104.0)
- added U13: ESP32-WROOM-32, RF_Module:ESP32-WROOM-32, F.Cu at (141.5, 85.1)
- added U14: CH340T, Package_SO:SSOP-20_5.3x7.2mm_P0.65mm, F.Cu at (152.1, 104.5)
- U11: value Olimex_ESP32-POE -> PCF8574; footprint Tales:Olimex_ESP32-POE_Pads -> Tales:SO-16_7.5x10.3mm_P1.27mm
- moved U11 14.0 mm to (133.3, 106.0)
Connections:
- U11 pad 1: +5V -> unconnected-(U11-Pad1)
- U11 pad 10: OUT8 -> unconnected-(U11-Pad10)
- U11 pad 11: OUT4 -> unconnected-(U11-Pad11)
- U11 pad 12: IN8 -> unconnected-(U11-Pad12)
- U11 pad 13: IN7 -> unconnected-(U11-Pad13)
- U11 pad 14: OUT3 -> unconnected-(U11-Pad14)
- U11 pad 15: OUT2 -> unconnected-(U11-Pad15)
- U11 pad 16: OUT1 -> unconnected-(U11-Pad16)
- U11 pad 3: GNDREF -> unconnected-(U11-Pad3)
- U11 pad 4: Net-(R35-Pad2) -> unconnected-(U11-Pad4)
- U11 pad 5: IN5 -> unconnected-(U11-Pad5)
- U11 pad 6: IN6 -> unconnected-(U11-Pad6)
- U11 pad 7: OUT5 -> unconnected-(U11-Pad7)
- U11 pad 8: OUT7 -> unconnected-(U11-Pad8)
- U11 pad 9: OUT6 -> unconnected-(U11-Pad9)
Routing:
- net OUT8: track 182.1 -> 11.6 mm, vias 2 -> 0
- net OUT7: track 163.0 -> 10.7 mm, vias 2 -> 0
- net OUT6: track 151.6 -> 9.83 mm, vias 2 -> 0
- net +24V: track 317.4 -> 184.7 mm, vias 2 -> 0
- net OUT5: track 132.5 -> 8.94 mm, vias 2 -> 0
- net OUT4: track 131.3 -> 8.04 mm, vias 2 -> 0
- net IN4: track 113.9 -> 0.00 mm, vias 4 -> 0
- net IN3: track 100.1 -> 0.00 mm, vias 4 -> 0
- net OUT3: track 107.1 -> 7.14 mm, vias 2 -> 0
- net IN8: track 94.8 -> 0.00 mm, vias 5 -> 0
- net IN7: track 92.3 -> 0.00 mm, vias 5 -> 0
- net IN2: track 87.0 -> 0.00 mm, vias 4 -> 0
- net OUT2: track 88.1 -> 6.24 mm, vias 2 -> 0
- net IN1: track 75.1 -> 0.00 mm, vias 3 -> 0
- net OUT1: track 68.5 -> 4.44 mm, vias 2 -> 0
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- removed copper zone on F.Cu, net +24V
Other:
- board text removed: "8x IN 24VDC/8x OUT RLY"
- board text removed: "ESP-RELAY-8CH-V1"
- board text removed: "MAX LOAD 10A/CHANNEL"
- board text removed: "OLIMEX ESP32-POE-ISO"
- board text removed: "TMASCHIO 2022"

Commit message: Development
Parts:
- removed the U14 at (152.1, 104.5)
- added C17: 10uF/16V/1206, Tales:C_1206_3216Metric, F.Cu at (169.5, 43.8)
- added C18: 0,1uF/50V/0805, Tales:C_0805_2012Metric, F.Cu at (168.9, 47.0)
- added D11: SS34, Tales:D_SMA, F.Cu at (132.1, 44.5)
- added D20: B5819W, Tales:D_SOD-123, F.Cu at (191.8, 49.5)
- added D31: B5819W, Tales:D_SOD-123, F.Cu at (150.2, 44.5)
- added F1: 500mA, Tales:Fuse_0402_1005Metric, F.Cu at (142.1, 44.5)
- added F1: 500mA, Tales:Fuse_0402_1005Metric, F.Cu at (190.3, 52.2)
- added J3: USB_B_Micro, Connector_USB:USB_Micro-B_Amphenol_10118194_Horizontal, F.Cu at (151.8, 129.3)
- added LOGO1: Logo_Open_Hardware_Large, Symbol:OSHW-Logo2_14.6x12mm_SilkScreen, F.Cu at (121.0, 48.2)
- added Q9: UMH3N, Package_TO_SOT_SMD:SOT-363_SC-70-6, F.Cu at (153.7, 118.1)
- added R50: 10k/0,125W/0805, Tales:R_0805_2012Metric, F.Cu at (168.9, 50.0)
- added R51: 10k/0,125W/0805, Tales:R_0805_2012Metric, F.Cu at (174.6, 43.6)
- added U12: CH340C, Package_SO:SOIC-16_3.9x9.9mm_P1.27mm, F.Cu at (152.4, 106.7)
- R22: renamed from R30; value 57,6k/0,125W/0805 -> 52,3k/0,125W/0805
- moved J12 4.44 mm to (140.3, 123.2)
- renumbered C8 to C10, C9 to C11, C10 to C12, C12 to C2, C2 to C3, C11 to C4, C3 to C5, C4 to C6, C5 to C7, C6 to C8, C7 to C9, D11 to D12, D12 to D13, D13 to D14, D14 to D15, D15 to D16, D16 to D17, D17 to D18, D18 to D19, D19 to D21, D20 to D22, D21 to D23, D22 to D24, D23 to D25, D24 to D26, D25 to D27, D26 to D28, D27 to D29, D28 to D30, D29 to D31, J9 to J10, J10 to J11, J11 to J12, J3 to J4, J4 to J5, J5 to J6, J6 to J7, J7 to J8, J8 to J9, R10 to R1, R8 to R10, R9 to R11, R20 to R12, R12 to R13, R13 to R14, R14 to R15, R15 to R16, R16 to R17, R17 to R18, R18 to R19, R11 to R2, R19 to R20, R29 to R21, R21 to R23, R22 to R24, R23 to R25, R24 to R26, R25 to R27, R26 to R28, R27 to R29, R1 to R3, R28 to R30, R36 to R35, R37 to R36, R38 to R37, R39 to R38, R40 to R39, R2 to R4, R41 to R40, R42 to R41, R43 to R42, R44 to R43, R45 to R44, R46 to R45, R47 to R46, R48 to R47, R49 to R48, R50 to R49, R3 to R5, R4 to R6, R5 to R7, R6 to R8, R7 to R9, U9 to U10, U12 to U14, U10 to U2, U2 to U3, U3 to U4, U4 to U5, U5 to U6, U6 to U7, U7 to U8, U8 to U9
Connections:
- C15 pad 1: +5V -> Net-(C15-Pad1)
- C16 pad 1: +5V -> Net-(C15-Pad1)
- L2 pad 2: +5V -> Net-(C15-Pad1)
- R21 pad 1: +5V -> Net-(C15-Pad1)
- U13 pad 1: Net-(U13-Pad1) -> GNDREF
- U13 pad 15: Net-(U13-Pad1) -> GNDREF
- U13 pad 2: unconnected-(U13-Pad2) -> +3.3V
- U13 pad 25: unconnected-(U13-Pad25) -> Net-(Q9-Pad6)
- U13 pad 3: unconnected-(U13-Pad3) -> Net-(Q9-Pad3)
- U13 pad 34: unconnected-(U13-Pad34) -> Net-(U12-Pad2)
- U13 pad 35: unconnected-(U13-Pad35) -> Net-(U12-Pad3)
- U13 pad 38: Net-(U13-Pad1) -> GNDREF
- U13 pad 39: Net-(U13-Pad1) -> GNDREF
- U14 pad 25: IN1 -> unconnected-(U14-Pad25)
Routing:
- net Net-(C15-Pad1): track 0.00 -> 128.7 mm, vias 0 -> 3
- net +5V: track 128.7 -> 0.00 mm, vias 3 -> 0
