File: V2/ESP-relay-8ch-V2.kicad_sch (KiCad schematic)
At the start: 143 parts, among them J1 +24VDC, J10 OUT8, J2 INPUTS, J3 OUT1, J4 OUT2, J5 OUT3, J6 OUT4, J7 OUT5, J8 OUT6, J9 OUT7, K1 G5PZ-1A, K2 G5PZ-1A, K3 G5PZ-1A, K4 G5PZ-1A, K5 G5PZ-1A, K6 G5PZ-1A, K7 G5PZ-1A, K8 G5PZ-1A, Q1 MMBT2222A/SOT-23-3, Q2 MMBT2222A/SOT-23-3, Q3 MMBT2222A/SOT-23-3, Q4 MMBT2222A/SOT-23-3, Q5 MMBT2222A/SOT-23-3, Q6 MMBT2222A/SOT-23-3, Q7 MMBT2222A/SOT-23-3, Q8 MMBT2222A/SOT-23-3, U1 SY8089A1AAC, U10 TX4138, U11 Olimex_ESP32-POE, U2 LTV-817S, U3 LTV-817S, U4 LTV-817S, U5 LTV-817S, U6 LTV-817S, U7 LTV-817S, U8 LTV-817S, U9 LTV-817S

Commit message: Dev
Parts:
- removed R35: 4k7/0,125W/0805, Tales:R_0805_2012Metric, symbol Device:R_US
- removed U11: Olimex_ESP32-POE, Tales:Olimex_ESP32-POE_Pads, symbol Tales:Olimex_ESP32-POE
Connections:
- no-connect marks 3 -> 2
Other:
- added sheet ESP32 (esp32.kicad_sch)

Commit message: Development
Parts:
- added D11: SS34, Tales:D_SMA, symbol Device:D_Schottky_Small
- added D20: B5819W, Tales:D_SOD-123, symbol Device:D_Schottky_Small
- added F1: 500mA, Tales:Fuse_0402_1005Metric, symbol Device:Fuse_Small
- added J3: USB_B_Micro, Connector_USB:USB_Micro-B_Amphenol_10118194_Horizontal, symbol Connector:USB_B_Micro
- D1: symbol Device:D -> Device:D_Small; Mfr MDD -> Microdiode; Technology (none) -> Rectifier
- D10: symbol Device:D_Schottky -> Device:D_Schottky_Small; Technology (none) -> Schottky
- D12: renamed from D11; symbol Device:LED -> Device:LED_Small
- D13: renamed from D12; symbol Device:LED -> Device:LED_Small
- D14: renamed from D13; symbol Device:LED -> Device:LED_Small
- D15: renamed from D14; symbol Device:LED -> Device:LED_Small
- D16: renamed from D15; symbol Device:D -> Device:D_Small
- D17: renamed from D16; symbol Device:D -> Device:D_Small
- D18: renamed from D17; symbol Device:D -> Device:D_Small
- D19: renamed from D18; symbol Device:D -> Device:D_Small
- D2, D3, D4, D5, D6, D7, D8, D9: symbol Device:D_Zener -> Device:D_Zener_Small
- D21: renamed from D19; symbol Device:LED -> Device:LED_Small
- D22: renamed from D20; symbol Device:LED -> Device:LED_Small
- D23: renamed from D21; symbol Device:LED -> Device:LED_Small
- D24: renamed from D22; symbol Device:LED -> Device:LED_Small
- D25: renamed from D23; symbol Device:LED -> Device:LED_Small
- D26: renamed from D24; symbol Device:D -> Device:D_Small
- D27: renamed from D25; symbol Device:D -> Device:D_Small
- D28: renamed from D26; symbol Device:D -> Device:D_Small
- D29: renamed from D27; symbol Device:D -> Device:D_Small
- D30: renamed from D28; symbol Device:LED -> Device:LED_Small
- D31: renamed from D29; symbol Device:LED -> Device:LED_Small
- R22: renamed from R30; value 57,6k/0,125W/0805 -> 52,3k/0,125W/0805; LCSC Part # C17758 -> C17740; Mfr PN 0805W8F5762T5E -> 0805W8F5232T5E; Vendor PN C17758 -> C17740
- renumbered C8 to C10, C9 to C11, C10 to C12, C12 to C2, C2 to C3, C11 to C4, C3 to C5, C4 to C6, C5 to C7, C6 to C8, C7 to C9, J9 to J10, J10 to J11, J3 to J4, J4 to J5, J5 to J6, J6 to J7, J7 to J8, J8 to J9, R10 to R1, R8 to R10, R9 to R11, R20 to R12, R12 to R13, R13 to R14, R14 to R15, R15 to R16, R16 to R17, R17 to R18, R18 to R19, R11 to R2, R19 to R20, R29 to R21, R21 to R23, R22 to R24, R23 to R25, R24 to R26, R25 to R27, R26 to R28, R27 to R29, R1 to R3, R28 to R30, R36 to R35, R37 to R36, R38 to R37, R39 to R38, R40 to R39, R2 to R4, R41 to R40, R42 to R41, R43 to R42, R44 to R43, R45 to R44, R46 to R45, R47 to R46, R48 to R47, R49 to R48, R50 to R49, R3 to R5, R4 to R6, R5 to R7, R6 to R8, R7 to R9, U9 to U10, U10 to U2, U2 to U3, U3 to U4, U4 to U5, U5 to U6, U6 to U7, U7 to U8, U8 to U9
Connections:
- net +5V: now also D11.1 (K), F1.2; no longer C15.1, C16.1, L2.2, R21.1
- net GNDREF: now also J3.5 (GND), J3.6 (Shield)
- new net: C15.1, C16.1, D11.2 (A), L2.2, R21.1
- new net: D20.1 (K), F1.1
- new net: D20.2 (A), J3.1 (VBUS)
- new net D+: J3.3 (D+)
- new net D-: J3.2 (D-)
- no-connect marks 2 -> 3
Other:
- note added: "5V MAIN"
- note added: "5V USB"
- moved on the sheet: C1, C13, C14, C15, C16, C2, C3, C4, D10, D12, D13, D14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
