File: V2/esp-relay-8ch-v2-inputs.kicad_sch (KiCad schematic)
At the start: 41 parts, among them J2 INPUTS, U10 LTV-817S, U11 LTV-817S, U4 LTV-817S, U5 LTV-817S, U6 LTV-817S, U7 LTV-817S, U8 LTV-817S, U9 LTV-817S

Commit message: Update to Kicad 8
Parts:
- renumbered R13 to R12, R15 to R13, R17 to R14, R19 to R15, R21 to R16, R23 to R17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
