File: V2/esp-relay-8ch-v2-outputs.kicad_sch (KiCad schematic)
At the start: 66 parts, among them J3 Conn_01x08, J4 Conn_01x08, K1 G5PZ-1A, K2 G5PZ-1A, K3 G5PZ-1A, K4 G5PZ-1A, K5 G5PZ-1A, K6 G5PZ-1A, K7 G5PZ-1A, K8 G5PZ-1A, Q1 MMBT2222A/SOT-23-3, Q2 MMBT2222A/SOT-23-3, Q3 MMBT2222A/SOT-23-3, Q4 MMBT2222A/SOT-23-3, Q5 MMBT2222A/SOT-23-3, Q6 MMBT2222A/SOT-23-3, Q7 MMBT2222A/SOT-23-3, Q8 MMBT2222A/SOT-23-3

Commit message: V2 design
Parts:
- D14, D16, D18, D20, D22, D24, D26, D28: value BLUE/0603 -> GREEN; LCSC Part # C72041 -> C72043; Mfr PN 19-217/BHC-ZL1M2RY/3T -> 19-217/GHC-YR1S2/3T; Package (none) -> 0603; Technology (none) -> InGaN; Vendor PN C72041 -> C72043
Changed lines of the file:
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@@
       (effects (font (size 1.27 1.27)) (justify left))
     )
-    (property "Value" "BLUE/0603" (at 97.79 72.39 90)
+    (property "Value" "GREEN" (at 97.79 72.39 90)
       (effects (font (size 1.27 1.27)) (justify left))
     )
@@
       (effects (font (size 1.27 1.27)) hide)
     )
-    (property "Mfr PN" "19-217/BHC-ZL1M2RY/3T" (at 100.33 72.39 0)
+    (property "Mfr PN" "19-217/GHC-YR1S2/3T" (at 100.33 72.39 0)
       (effects (font (size 1.27 1.27)) hide)
     )
-    (property "Technology" "~" (at 100.33 72.39 0)
+    (property "Technology" "InGaN" (at 100.33 72.39 0)
       (effects (font (size 1.27 1.27)) hide)
     )
@@
       (effects (font (size 1.27 1.27)) hide)
     )
-    (property "Vendor PN" "C72041" (at 100.33 72.39 0)
+    (property "Vendor PN" "C72043" (at 100.33 72.39 0)
       (effects (font (size 1.27 1.27)) hide)
     )
-    (property "LCSC Part #" "C72041" (at 97.79 74.93 90)
+    (property "LCSC Part #" "C72043" (at 97.79 74.93 90)
       (effects (font (size 1.27 1.27)) (justify left))
     )
@@
       (effects (font (size 1.27 1.27)) hide)
     )
+    (property "Package" "0603" (at 100.33 72.39 0)
+      (effects (font (size 1.27 1.27)) hide)
+    )
     (pin "1")
     (pin "2")
@@
       (effects (font (size 1.27 1.27)) (justify left))
     )
-    (property "Value" "BLUE/0603" (at 226.06 115.57 90)
+    (property "Value" "GREEN" (at 226.06 115.57 90)
       (effects (font (size 1.27 1.27)) (justify left))
     )
@@
       (effects (font (size 1.27 1.27)) hide)
     )
-    (property "Mfr PN" "19-217/BHC-ZL1M2RY/3T" (at 228.6 115.57 0)
+    (property "Mfr PN" "19-217/GHC-YR1S2/3T" (at 228.6 115.57 0)
       (effects (font (size 1.27 1.27)) hide)
     )
-    (property "Technology" "~" (at 228.6 115.57 0)
+    (property "Technology" "InGaN" (at 228.6 115.57 0)
       (effects (font (size 1.27 1.27)) hide)
     )
@@
       (effects (font (size 1.27 1.27)) hide)
     )
-    (property "Vendor PN" "C72041" (at 228.6 115.57 0)
+    (property "Vendor PN" "C72043" (at 228.6 115.57 0)
       (effects (font (size 1.27 1.27)) hide)
     )
-    (property "LCSC Part #" "C72041" (at 226.06 118.11 90)
+    (property "LCSC Part #" "C72043" (at 226.06 118.11 90)
       (effects (font (size 1.27 1.27)) (justify left))
     )
@@
       (effects (font (size 1.27 1.27)) hide)
     )
+    (property "Package" "0603" (at 228.6 115.57 0)
+      (effects (font (size 1.27 1.27)) hide)
+    )
     (pin "1")
     (pin "2")
@@
       (effects (font (size 1.27 1.27)) (justify left))
     )
-    (property "Value" "BLUE/0603" (at 97.79 158.75 90)
+    (property "Value" "GREEN" (at 97.79 158.75 90)
       (effects (font (size 1.27 1.27)) (justify left))
     )
@@
       (effects (font (size 1.27 1.27)) hide)
     )
-    (property "Mfr PN" "19-217/BHC-ZL1M2RY/3T" (at 100.33 158.75 0)
+    (property "Mfr PN" "19-217/GHC-YR1S2/3T" (at 100.33 158.75 0)
       (effects (font (size 1.27 1.27)) hide)
     )
-    (property "Technology" "~" (at 100.33 158.75 0)
+    (property "Technology" "InGaN" (at 100.33 158.75 0)
       (effects (font (size 1.27 1.27)) hide)
     )
@@
       (effects (font (size 1.27 1.27)) hide)
     )
-    (property "Vendor PN" "C72041" (at 100.33 158.75 0)
+    (property "Vendor PN" "C72043" (at 100.33 158.75 0)
       (effects (font (size 1.27 1.27)) hide)
     )
-    (property "LCSC Part #" "C72041" (at 97.79 161.29 90)
+    (property "LCSC Part #" "C72043" (at 97.79 161.29 90)
       (effects (font (size 1.27 1.27)) (justify left))
     )
@@
       (effects (font (size 1.27 1.27)) hide)
     )
+    (property "Package" "0603" (at 100.33 158.75 0)
+      (effects (font (size 1.27 1.27)) hide)
+    )
     (pin "1")
     (pin "2")
@@
       (effects (font (size 1.27 1.27)) (justify left))
     )
-    (property "Value" "BLUE/0603" (at 97.79 201.93 90)
+    (property "Value" "GREEN" (at 97.79 201.93 90)
       (effects (font (size 1.27 1.27)) (justify left))
     )
@@
       (effects (font (size 1.27 1.27)) hide)
     )
-    (property "Mfr PN" "19-217/BHC-ZL1M2RY/3T" (at 100.33 201.93 0)
+    (property "Mfr PN" "19-217/GHC-YR1S2/3T" (at 100.33 201.93 0)
       (effects (font (size 1.27 1.27)) hide)
     )
-    (property "Technology" "~" (at 100.33 201.93 0)
+    (property "Technology" "InGaN" (at 100.33 201.93 0)
       (effects (font (size 1.27 1.27)) hide)
     )
@@
       (effects (font (size 1.27 1.27)) hide)
     )
-    (property "Vendor PN" "C72041" (at 100.33 201.93 0)
+    (property "Vendor PN" "C72043" (at 100.33 201.93 0)
       (effects (font (size 1.27 1.27)) hide)
     )
-    (property "LCSC Part #" "C72041" (at 97.79 204.47 90)
+    (property "LCSC Part #" "C72043" (at 97.79 204.47 90)
       (effects (font (size 1.27 1.27)) (justify left))
     )
@@
       (effects (font (size 1.27 1.27)) hide)
     )
+    (property "Package" "0603" (at 100.33 201.93 0)
+      (effects (font (size 1.27 1.27)) hide)
+    )
     (pin "1")
     (pin "2")
@@
       (effects (font (size 1.27 1.27)) (justify left))
     )
-    (property "Value" "BLUE/0603" (at 226.06 201.93 90)
+    (property "Value" "GREEN" (at 226.06 201.93 90)
       (effects (font (size 1.27 1.27)) (justify left))
     )
@@
       (effects (font (size 1.27 1.27)) hide)
     )
-    (property "Mfr PN" "19-217/BHC-ZL1M2RY/3T" (at 228.6 201.93 0)
+    (property "Mfr PN" "19-217/GHC-YR1S2/3T" (at 228.6 201.93 0)
       (effects (font (size 1.27 1.27)) hide)
     )
-    (property "Technology" "~" (at 228.6 201.93 0)
+    (property "Technology" "InGaN" (at 228.6 201.93 0)
       (effects (font (size 1.27 1.27)) hide)
     )
@@
       (effects (font (size 1.27 1.27)) hide)
     )
-    (property "Vendor PN" "C72041" (at 228.6 201.93 0)
+    (property "Vendor PN" "C72043" (at 228.6 201.93 0)
       (effects (font (size 1.27 1.27)) hide)
     )
-    (property "LCSC Part #" "C72041" (at 226.06 204.47 90)
+    (property "LCSC Part #" "C72043" (at 226.06 204.47 90)
       (effects (font (size 1.27 1.27)) (justify left))
     )
@@
       (effects (font (size 1.27 1.27)) hide)
     )
+    (property "Package" "0603" (at 228.6 201.93 0)
+      (effects (font (size 1.27 1.27)) hide)
+    )
     (pin "1")
     (pin "2")
@@
       (effects (font (size 1.27 1.27)) (justify left))
     )
-    (property "Value" "BLUE/0603" (at 226.06 72.39 90)
+    (property "Value" "GREEN" (at 226.06 72.39 90)
       (effects (font (size 1.27 1.27)) (justify left))
     )
@@
       (effects (font (size 1.27 1.27)) hide)
     )
-    (property "Mfr PN" "19-217/BHC-ZL1M2RY/3T" (at 228.6 72.39 0)
+    (property "Mfr PN" "19-217/GHC-YR1S2/3T" (at 228.6 72.39 0)
       (effects (font (size 1.27 1.27)) hide)
     )
-    (property "Technology" "~" (at 228.6 72.39 0)
+    (property "Technology" "InGaN" (at 228.6 72.39 0)
       (effects (font (size 1.27 1.27)) hide)
     )
@@
       (effects (font (size 1.27 1.27)) hide)
     )
-    (property "Vendor PN" "C72041" (at 228.6 72.39 0)
+    (property "Vendor PN" "C72043" (at 228.6 72.39 0)
       (effects (font (size 1.27 1.27)) hide)
     )
-    (property "LCSC Part #" "C72041" (at 226.06 74.93 90)
+    (property "LCSC Part #" "C72043" (at 226.06 74.93 90)
       (effects (font (size 1.27 1.27)) (justify left))
     )
@@
       (effects (font (size 1.27 1.27)) hide)
     )
+    (property "Package" "0603" (at 228.6 72.39 0)
+      (effects (font (size 1.27 1.27)) hide)
+    )
     (pin "1")
     (pin "2")
@@
       (effects (font (size 1.27 1.27)) (justify left))
     )
-    (property "Value" "BLUE/0603" (at 97.79 115.57 90)
+    (property "Value" "GREEN" (at 97.79 115.57 90)
       (effects (font (size 1.27 1.27)) (justify left))
     )
@@
       (effects (font (size 1.27 1.27)) hide)
     )
-    (property "Mfr PN" "19-217/BHC-ZL1M2RY/3T" (at 100.33 115.57 0)
+    (property "Mfr PN" "19-217/GHC-YR1S2/3T" (at 100.33 115.57 0)
       (effects (font (size 1.27 1.27)) hide)
     )
-    (property "Technology" "~" (at 100.33 115.57 0)
+    (property "Technology" "InGaN" (at 100.33 115.57 0)
       (effects (font (size 1.27 1.27)) hide)
     )
@@
       (effects (font (size 1.27 1.27)) hide)
     )
-    (property "Vendor PN" "C72041" (at 100.33 115.57 0)
+    (property "Vendor PN" "C72043" (at 100.33 115.57 0)
       (effects (font (size 1.27 1.27)) hide)
     )
-    (property "LCSC Part #" "C72041" (at 97.79 118.11 90)
+    (property "LCSC Part #" "C72043" (at 97.79 118.11 90)
       (effects (font (size 1.27 1.27)) (justify left))
     )
@@
       (effects (font (size 1.27 1.27)) hide)
     )
+    (property "Package" "0603" (at 100.33 115.57 0)
+      (effects (font (size 1.27 1.27)) hide)
+    )
     (pin "1")
     (pin "2")
@@
       (effects (font (size 1.27 1.27)) (justify left))
     )
-    (property "Value" "BLUE/0603" (at 226.06 158.75 90)
+    (property "Value" "GREEN" (at 226.06 158.75 90)
       (effects (font (size 1.27 1.27)) (justify left))
     )
@@
       (effects (font (size 1.27 1.27)) hide)
     )
-    (property "Mfr PN" "19-217/BHC-ZL1M2RY/3T" (at 228.6 158.75 0)
+    (property "Mfr PN" "19-217/GHC-YR1S2/3T" (at 228.6 158.75 0)
       (effects (font (size 1.27 1.27)) hide)
     )
-    (property "Technology" "~" (at 228.6 158.75 0)
+    (property "Technology" "InGaN" (at 228.6 158.75 0)
       (effects (font (size 1.27 1.27)) hide)
     )
@@
       (effects (font (size 1.27 1.27)) hide)
     )
-    (property "Vendor PN" "C72041" (at 228.6 158.75 0)
+    (property "Vendor PN" "C72043" (at 228.6 158.75 0)
       (effects (font (size 1.27 1.27)) hide)
     )
-    (property "LCSC Part #" "C72041" (at 226.06 161.29 90)
+    (property "LCSC Part #" "C72043" (at 226.06 161.29 90)
       (effects (font (size 1.27 1.27)) (justify left))
     )
@@
       (effects (font (size 1.27 1.27)) hide)
     )
+    (property "Package" "0603" (at 228.6 158.75 0)
+      (effects (font (size 1.27 1.27)) hide)
+    )

Commit message: Update to Kicad 8
Parts:
- renumbered D16 to D15, D18 to D16, D20 to D17, D15 to D18, D17 to D19, D19 to D20, D24 to D23, D26 to D24, D28 to D25, D23 to D26, D25 to D27, D27 to D28, R30 to R29, R31 to R30, R33 to R31, R34 to R32, R36 to R33, R37 to R34, R29 to R35, R32 to R36, R35 to R37, R42 to R41, R43 to R42, R45 to R43, R46 to R44, R48 to R45, R49 to R46, R41 to R47, R44 to R48, R47 to R49
