File: V2/esp-relay-8ch-v2.kicad_sch (KiCad schematic)
At the start: 23 parts, among them J1 +24VDC, U1 TX4138, U2 SY8089A1AAC

Commit message: V2 design
Parts:
- removed C6, C8: 10uF/16V/1206, Tales:C_1206_3216Metric, symbol Device:C_Polarized_Small_US
- removed D1: SM4007PL/SOD-123, Tales:D_SOD-123, symbol Device:D
- removed D4: BLUE/0603, Tales:LED_0603_1608Metric, symbol Device:LED
- added C17, C8: 22uF/10V, Tales:C_1206_3216Metric, symbol Device:C_Small
- added C6: 10uF/10V, Tales:C_0603_1608Metric, symbol Device:C_Small
- added D1: SS34, Tales:D_SMA, symbol Device:D_Schottky_Small
- added D3: GREEN, Tales:LED_0603_1608Metric, symbol Device:LED_Small
- C3: value 0,1uF/50V/0805 -> 100nF/100V; Case 0805/2012 -> (none); LCSC Part # C49678 -> C28233; Mfr Yageo -> Samsung; Mfr PN CC0805KRX7R9BB104 -> CL21B104KCFNNNE; Package (none) -> 0805/2012; Technology Ceramic -> Ceramix X7R; Vendor PN C49678 -> C28233
- C5: value 470uF/16V/10x10 -> 470uF/16V; footprint Tales:CP_Elec_10x10 -> Tales:CP_Elec_8x10.5; Case 10x10 -> (none); LCSC Part # C249930 -> C96179; Mfr Lelon -> Semtech; Mfr PN VZH471M1CTR-1010 -> CS1C471M-CRF10; Package (none) -> D8xL10.5mm; Vendor PN C249930 -> C96179
- C7: value 22pF/50V/0603 -> 22pF/50V; footprint Tales:C_0603_1608Metric -> Tales:C_0402_1005Metric; Case 0603/1608 -> (none); LCSC Part # C1653 -> C1555; Mfr Samsung -> FH; Mfr PN CL10C220JB8NNNC -> 0402CG220J500NT; Package (none) -> 0402/1005; Technology Ceramic -> Ceramic C0G; Vendor PN C1653 -> C1555
- R2: value 5R1/0,125W/0805 -> 5,1R/100mW; footprint Tales:R_0805_2012Metric -> Tales:R_0603_1608Metric; Case 0805/2012 -> (none); LCSC Part # C17724 -> C25197; Mfr Uniroyal -> UNI-ROYAL(Uniroyal Elec); Mfr PN 0805W8F510KT5E -> 0603WAF510KT5E; Package (none) -> 0603/1608; Technology (none) -> 1%; Vendor PN C17724 -> C25197
- R3: value 300k/0,125W/0805 -> 300k/100mW; footprint Tales:R_0805_2012Metric -> Tales:R_0603_1608Metric; Case 0805/2012 -> (none); LCSC Part # C17616 -> C23024; Mfr Uniroyal -> UNI-ROYAL(Uniroyal Elec); Mfr PN 0805W8F3003T5E -> 0603WAF3003T5E; Package (none) -> 0603/1608; Technology (none) -> 1%; Vendor PN C17616 -> C23024
- R4: value 57,6k/0,125W/0805 -> 52,3k/100mW; footprint Tales:R_0805_2012Metric -> Tales:R_0603_1608Metric; Case 0805/2012 -> (none); LCSC Part # C17758 -> C185323; Mfr Uniroyal -> Yageo; Mfr PN 0805W8F5762T5E -> RC0603FR-0752K3L; Package (none) -> 0603/1608; Technology (none) -> 1%; Vendor PN C17758 -> C185323
- R7: value 820R/0,125W/0805 -> 820R/100mW; footprint Tales:R_0805_2012Metric -> Tales:R_0603_1608Metric; Case 0805/2012 -> (none); LCSC Part # C17837 -> C23253; Mfr Uniroyal -> UNI-ROYAL(Uniroyal Elec); Mfr PN 0805W8F8200T5E -> 0603WAF8200T5E; Package (none) -> 0603/1608; Technology (none) -> 1%; Vendor PN C17837 -> C23253
Connections:
- net +24V: now also D1.2 (A)
- net +3.3V: now also C17.1, C8.1
- net +5V: now also C6.1
- net GNDREF: now also C17.2, C6.2, C8.2, D3.1 (K)
- net at C1.1, C2.1, R1.1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: now also D1.1 (K)
- net at R7.2: now also D3.2 (A)
